File: SCI-BREADBRD_sci_conn.sch (KiCad schematic (older format))
At the start: 6 parts

Commit message: Fixed the footprint properties of various parts throughout the schematic to make sure they are all point to valid footprints.
Added SCI-BREADBRD.cmp to specify which footprints should be used for
each part.

Added netlists to the .gitignore as those can be generated easily in
eeschema.
Parts:
- P4: renamed from P?; footprint QRM8-026-02_0-L-D-A -> SAMTEC_QRM8-026-02_0-L-D-A
- gave numbers to parts that had none: 5
Changed lines of the file:
@@
-EESchema Schematic File Version 2  date Fri 27 Apr 2012 04:22:34 AM EDT
+EESchema Schematic File Version 2  date Fri 27 Apr 2012 08:55:37 AM EDT
 LIBS:custom_transistors
 LIBS:TI_custom
@@
 $EndDescr
 $Comp
-L MARK_SCI_CONN P?
+L MARK_SCI_CONN P4
 U 1 1 4F9A652C
 P 3700 4200
-F 0 "P?" H 4600 7050 60  0000 C CNN
+F 0 "P4" H 4600 7050 60  0000 C CNN
 F 1 "MARK_SCI_CONN" H 3750 7050 60  0000 C CNN
-F 2 "QRM8-026-02_0-L-D-A" H 3700 4200 60  0001 C CNN
+F 2 "SAMTEC_QRM8-026-02_0-L-D-A" H 3700 4200 60  0001 C CNN
 F 4 "SAMTEC" H 3700 4200 60  0001 C CNN "Manufacturer"
 F 5 "QRM8-026-02.0-L-D-A" H 3700 4200 60  0001 C CNN "Part Number"
@@
 $EndComp
 $Comp
-L CONN_16 P?
+L CONN_16 P5
 U 1 1 4F9A6535
 P 5950 4850
-F 0 "P?" H 5950 5750 60  0000 C CNN
+F 0 "P5" H 5950 5750 60  0000 C CNN
 F 1 "CONN_16" H 6000 4050 60  0000 C CNN
 F 2 "PIN_ARRAY_1x16" H 5950 4850 60  0001 C CNN
@@
 $EndComp
 $Comp
-L GND #PWR?
+L GND #PWR014
 U 1 1 4F9A653B
 P 2250 6500
-F 0 "#PWR?" H 2250 6500 30  0001 C CNN
+F 0 "#PWR014" H 2250 6500 30  0001 C CNN
 F 1 "GND" H 2250 6430 30  0001 C CNN
 	1    2250 6500
@@
 $EndComp
 $Comp
-L GND #PWR?
+L GND #PWR015
 U 1 1 4F9A6541
 P 5150 2950
-F 0 "#PWR?" H 5150 2950 30  0001 C CNN
+F 0 "#PWR015" H 5150 2950 30  0001 C CNN
 F 1 "GND" H 5150 2880 30  0001 C CNN
 	1    5150 2950
@@
 $EndComp
 $Comp
-L GND #PWR?
+L GND #PWR016
 U 1 1 4F9A6547
 P 5150 2200
-F 0 "#PWR?" H 5150 2200 30  0001 C CNN
+F 0 "#PWR016" H 5150 2200 30  0001 C CNN
 F 1 "GND" H 5150 2130 30  0001 C CNN
 	1    5150 2200
@@
 $EndComp
 $Comp
-L GND #PWR?
+L GND #PWR017
 U 1 1 4F9A654D
 P 2250 2200
-F 0 "#PWR?" H 2250 2200 30  0001 C CNN
+F 0 "#PWR017" H 2250 2200 30  0001 C CNN
 F 1 "GND" H 2250 2130 30  0001 C CNN
 	1    2250 2200
@@
 $EndComp
 $Comp
-L GND #PWR?
+L GND #PWR018
 U 1 1 4F9A6553
 P 2250 2950
-F 0 "#PWR?" H 2250 2950 30  0001 C CNN
+F 0 "#PWR018" H 2250 2950 30  0001 C CNN
 F 1 "GND" H 2250 2880 30  0001 C CNN
 	1    2250 2950
@@
 $EndComp
 $Comp
-L GND #PWR?
+L GND #PWR019
 U 1 1 4F9A6559
 P 2250 3400
-F 0 "#PWR?" H 2250 3400 30  0001 C CNN
+F 0 "#PWR019" H 2250 3400 30  0001 C CNN
 F 1 "GND" H 2250 3330 30  0001 C CNN
 	1    2250 3400
@@
 $EndComp
 $Comp
-L GND #PWR?
+L GND #PWR020
 U 1 1 4F9A655F
 P 2250 3850
-F 0 "#PWR?" H 2250 3850 30  0001 C CNN
+F 0 "#PWR020" H 2250 3850 30  0001 C CNN
 F 1 "GND" H 2250 3780 30  0001 C CNN
 	1    2250 3850
@@
 $EndComp
 $Comp
-L GND #PWR?
+L GND #PWR021
 U 1 1 4F9A6565
 P 2250 4600
-F 0 "#PWR?" H 2250 4600 30  0001 C CNN
+F 0 "#PWR021" H 2250 4600 30  0001 C CNN
 F 1 "GND" H 2250 4530 30  0001 C CNN
 	1    2250 4600
@@
 $EndComp
 $Comp
-L GND #PWR?
+L GND #PWR022
 U 1 1 4F9A656B
 P 2250 5050
-F 0 "#PWR?" H 2250 5050 30  0001 C CNN
+F 0 "#PWR022" H 2250 5050 30  0001 C CNN
 F 1 "GND" H 2250 4980 30  0001 C CNN
 	1    2250 5050
@@
 $EndComp
 $Comp
-L GND #PWR?
+L GND #PWR023
 U 1 1 4F9A6571
 P 2250 5350
-F 0 "#PWR?" H 2250 5350 30  0001 C CNN
+F 0 "#PWR023" H 2250 5350 30  0001 C CNN
 F 1 "GND" H 2250 5280 30  0001 C CNN
 	1    2250 5350
@@
 $EndComp
 $Comp
-L GND #PWR?
+L GND #PWR024
 U 1 1 4F9A6577
 P 2250 5650
-F 0 "#PWR?" H 2250 5650 30  0001 C CNN
+F 0 "#PWR024" H 2250 5650 30  0001 C CNN
 F 1 "GND" H 2250 5580 30  0001 C CNN
 	1    2250 5650
@@
 MOD_IRQ
 $Comp
-L R_US R?
+L R_US R4
 U 1 1 4F9A6590
 P 1700 3950
-F 0 "R?" H 1700 4050 50  0000 C CNN
+F 0 "R4" H 1700 4050 50  0000 C CNN
 F 1 "0.10" H 1700 3850 50  0000 C CNN
 F 2 "SM0805" H 1700 3950 60  0001 C CNN
@@
 $EndComp
 $Comp
-L SCI_AVDD_5_5V #PWR?
+L SCI_AVDD_5_5V #PWR025
 U 1 1 4F9A6596
 P 1350 3850
-F 0 "#PWR?" H 1350 3950 30  0001 C CNN
+F 0 "#PWR025" H 1350 3950 30  0001 C CNN
 F 1 "SCI_AVDD_5_5V" H 1350 3950 30  0000 C CNN
 	1    1350 3850
@@
 $EndComp
 $Comp
-L R_US R?
+L R_US R3
 U 1 1 4F9A659F
 P 1200 4250
-F 0 "R?" H 1200 4350 50  0000 C CNN
+F 0 "R3" H 1200 4350 50  0000 C CNN
 F 1 "0.10" H 1200 4150 50  0000 C CNN
 F 2 "SM0805" H 1200 4250 60  0001 C CNN
@@
 $EndComp
 $Comp
-L AFE/SCI_ANLG_VDD #PWR?
+L AFE/SCI_ANLG_VDD #PWR026
 U 1 1 4F9A65A5
 P 1850 5700
-F 0 "#PWR?" H 1850 5800 30  0001 C CNN
+F 0 "#PWR026" H 1850 5800 30  0001 C CNN
 F 1 "AFE/SCI_ANLG_VDD" H 1850 5800 30  0000 C CNN
 	1    1850 5700
@@
 $EndComp
 $Comp
-L AFE/SCI_ANLG_VSS #PWR?
+L AFE/SCI_ANLG_VSS #PWR027
 U 1 1 4F9A65AB
 P 1850 5950
-F 0 "#PWR?" H 1850 5850 30  0001 C CNN
+F 0 "#PWR027" H 1850 5850 30  0001 C CNN
 F 1 "AFE/SCI_ANLG_VSS" H 1850 5850 30  0000 C CNN
 	1    1850 5950
@@
 SCI_PWR_GOOD
 $Comp
-L AFE/SCI_VREF_VDD #PWR?
+L AFE/SCI_VREF_VDD #PWR028
 U 1 1 4F9A65B2
 P 1850 4650
-F 0 "#PWR?" H 1850 4750 30  0001 C CNN
+F 0 "#PWR028" H 1850 4750 30  0001 C CNN
 F 1 "AFE/SCI_VREF_VDD" H 1850 4750 30  0000 C CNN
 	1    1850 4650
@@
 $EndComp
 $Comp
-L AFE/SCI_VREF_VSS #PWR?
+L AFE/SCI_VREF_VSS #PWR029
 U 1 1 4F9A65B8
 P 1850 4900
-F 0 "#PWR?" H 1850 4800 30  0001 C CNN
+F 0 "#PWR029" H 1850 4800 30  0001 C CNN
 F 1 "AFE/SCI_VREF_VSS" H 1850 4800 30  0000 C CNN
 	1    1850 4900
@@
 AFE/SCI_VREF
 $Comp
-L AFE/SCI_VREF_VSS #PWR?
+L AFE/SCI_VREF_VSS #PWR030
 U 1 1 4F9A65BF
 P 9300 4350
-F 0 "#PWR?" H 9300 4250 30  0001 C CNN
+F 0 "#PWR030" H 9300 4250 30  0001 C CNN
 F 1 "AFE/SCI_VREF_VSS" H 9300 4250 30  0000 C CNN
 	1    9300 4350
@@
 $EndComp
 $Comp
-L AFE/SCI_ANLG_VSS #PWR?
+L AFE/SCI_ANLG_VSS #PWR031
 U 1 1 4F9A65C5
 P 8800 4350
-F 0 "#PWR?" H 8800 4250 30  0001 C CNN
+F 0 "#PWR031" H 8800 4250 30  0001 C CNN
 F 1 "AFE/SCI_ANLG_VSS" H 8800 4250 30  0000 C CNN
 	1    8800 4350
@@
 $EndComp
 $Comp
-L AFE/SCI_ANLG_VDD #PWR?
+L AFE/SCI_ANLG_VDD #PWR032
 U 1 1 4F9A65CB
 P 8800 3200
-F 0 "#PWR?" H 8800 3300 30  0001 C CNN
+F 0 "#PWR032" H 8800 3300 30  0001 C CNN
 F 1 "AFE/SCI_ANLG_VDD" H 8800 3300 30  0000 C CNN
 	1    8800 3200
@@
 $EndComp
 $Comp
-L SCI_AVDD_5_5V #PWR?
+L SCI_AVDD_5_5V #PWR033
 U 1 1 4F9A65D1
 P 8250 3200
-F 0 "#PWR?" H 8250 3300 30  0001 C CNN
+F 0 "#PWR033" H 8250 3300 30  0001 C CNN
 F 1 "SCI_AVDD_5_5V" H 8250 3300 30  0000 C CNN
 	1    8250 3200
@@
 $EndComp
 $Comp
-L GND #PWR?
+L GND #PWR034
 U 1 1 4F9A65D7
 P 9650 4200
-F 0 "#PWR?" H 9650 4200 30  0001 C CNN
+F 0 "#PWR034" H 9650 4200 30  0001 C CNN
 F 1 "GND" H 9650 4130 30  0001 C CNN
 	1    9650 4200
@@
 AFE/SCI_VREF
 $Comp
-L AFE/SCI_VREF_VDD #PWR?
+L AFE/SCI_VREF_VDD #PWR035
 U 1 1 4F9A65DF
 P 9300 3200
-F 0 "#PWR?" H 9300 3300 30  0001 C CNN
+F 0 "#PWR035" H 9300 3300 30  0001 C CNN
 F 1 "AFE/SCI_VREF_VDD" H 9300 3300 30  0000 C CNN
 	1    9300 3200
@@
 $EndComp
 $Comp
-L GND #PWR?
+L GND #PWR036
 U 1 1 4F9A65E5
 P 9650 3350
-F 0 "#PWR?" H 9650 3350 30  0001 C CNN
+F 0 "#PWR036" H 9650 3350 30  0001 C CNN
 F 1 "GND" H 9650 3280 30  0001 C CNN
 	1    9650 3350
@@
 $EndComp
 $Comp
-L CONN_8X2 P?
+L CONN_8X2 P6
 U 1 1 4F9A65EE
 P 6100 3350
-F 0 "P?" H 6150 4250 60  0000 C CNN
+F 0 "P6" H 6150 4250 60  0000 C CNN
 F 1 "CONN_8X2" H 6150 3350 60  0000 C CNN
 F 2 "PIN_ARRAY_2x8" H 6100 3350 60  0001 C CNN
@@
 $EndComp
 $Comp
-L GND #PWR?
+L GND #PWR037
 U 1 1 4F9A65F4
 P 5150 6500
-F 0 "#PWR?" H 5150 6500 30  0001 C CNN
+F 0 "#PWR037" H 5150 6500 30  0001 C CNN
 F 1 "GND" H 5150 6430 30  0001 C CNN
 	1    5150 6500
@@
 $EndComp
 $Comp
-L CONN_8X2 P?
+L CONN_8X2 P7
 U 1 1 4F9A65FD
 P 9600 3700
-F 0 "P?" V 9560 4150 60  0000 C CNN
+F 0 "P7" V 9560 4150 60  0000 C CNN
 F 1 "CONN_8X2" V 9680 4150 60  0000 C CNN
 F 2 "PIN_ARRAY_2x8" H 9600 3700 60  0001 C CNN
@@
 $EndComp
 $Comp
-L SCI_DVDD_3_3V #PWR?
+L SCI_DVDD_3_3V #PWR038
 U 1 1 4F9A6603
 P 850 4150
-F 0 "#PWR?" H 850 4250 30  0001 C CNN
+F 0 "#PWR038" H 850 4250 30  0001 C CNN
 F 1 "SCI_DVDD_3_3V" H 850 4250 30  0000 C CNN
 	1    850  4150
@@
 $EndComp
 $Comp
-L SCI_DVDD_3_3V #PWR?
+L SCI_DVDD_3_3V #PWR039
 U 1 1 4F9A6609
 P 8400 4000
-F 0 "#PWR?" H 8400 4100 30  0001 C CNN
+F 0 "#PWR039" H 8400 4100 30  0001 C CNN
 F 1 "SCI_DVDD_3_3V" H 8400 4100 30  0000 C CNN
 	1    8400 4000
