File: SCI-BREADBRD_sci_conn.sch (KiCad schematic (older format))
At the start: 6 parts, among them P4 MARK_SCI_CONN, P5 CONN_16, P6 CONN_8X2, P7 CONN_8X2

Commit message: Completed ERC. Added some power flags and fixed mis-connected pins.
Changed lines of the file:
@@
-EESchema Schematic File Version 2  date Fri 27 Apr 2012 09:11:54 AM EDT
+EESchema Schematic File Version 2  date Fri 27 Apr 2012 11:11:24 AM EDT
 LIBS:custom_transistors
 LIBS:TI_custom
@@
 $EndComp
 $Comp
-L GND #PWR014
+L GND #PWR016
 U 1 1 4F9A653B
 P 2250 6500
-F 0 "#PWR014" H 2250 6500 30  0001 C CNN
+F 0 "#PWR016" H 2250 6500 30  0001 C CNN
 F 1 "GND" H 2250 6430 30  0001 C CNN
 	1    2250 6500
@@
 $EndComp
 $Comp
-L GND #PWR015
+L GND #PWR017
 U 1 1 4F9A6541
 P 5150 2950
-F 0 "#PWR015" H 5150 2950 30  0001 C CNN
+F 0 "#PWR017" H 5150 2950 30  0001 C CNN
 F 1 "GND" H 5150 2880 30  0001 C CNN
 	1    5150 2950
@@
 $EndComp
 $Comp
-L GND #PWR016
+L GND #PWR018
 U 1 1 4F9A6547
 P 5150 2200
-F 0 "#PWR016" H 5150 2200 30  0001 C CNN
+F 0 "#PWR018" H 5150 2200 30  0001 C CNN
 F 1 "GND" H 5150 2130 30  0001 C CNN
 	1    5150 2200
@@
 $EndComp
 $Comp
-L GND #PWR017
+L GND #PWR019
 U 1 1 4F9A654D
 P 2250 2200
-F 0 "#PWR017" H 2250 2200 30  0001 C CNN
+F 0 "#PWR019" H 2250 2200 30  0001 C CNN
 F 1 "GND" H 2250 2130 30  0001 C CNN
 	1    2250 2200
@@
 $EndComp
 $Comp
-L GND #PWR018
+L GND #PWR020
 U 1 1 4F9A6553
 P 2250 2950
-F 0 "#PWR018" H 2250 2950 30  0001 C CNN
+F 0 "#PWR020" H 2250 2950 30  0001 C CNN
 F 1 "GND" H 2250 2880 30  0001 C CNN
 	1    2250 2950
@@
 $EndComp
 $Comp
-L GND #PWR019
+L GND #PWR021
 U 1 1 4F9A6559
 P 2250 3400
-F 0 "#PWR019" H 2250 3400 30  0001 C CNN
+F 0 "#PWR021" H 2250 3400 30  0001 C CNN
 F 1 "GND" H 2250 3330 30  0001 C CNN
 	1    2250 3400
@@
 $EndComp
 $Comp
-L GND #PWR020
+L GND #PWR022
 U 1 1 4F9A655F
 P 2250 3850
-F 0 "#PWR020" H 2250 3850 30  0001 C CNN
+F 0 "#PWR022" H 2250 3850 30  0001 C CNN
 F 1 "GND" H 2250 3780 30  0001 C CNN
 	1    2250 3850
@@
 $EndComp
 $Comp
-L GND #PWR021
+L GND #PWR023
 U 1 1 4F9A6565
 P 2250 4600
-F 0 "#PWR021" H 2250 4600 30  0001 C CNN
+F 0 "#PWR023" H 2250 4600 30  0001 C CNN
 F 1 "GND" H 2250 4530 30  0001 C CNN
 	1    2250 4600
@@
 $EndComp
 $Comp
-L GND #PWR022
+L GND #PWR024
 U 1 1 4F9A656B
 P 2250 5050
-F 0 "#PWR022" H 2250 5050 30  0001 C CNN
+F 0 "#PWR024" H 2250 5050 30  0001 C CNN
 F 1 "GND" H 2250 4980 30  0001 C CNN
 	1    2250 5050
@@
 $EndComp
 $Comp
-L GND #PWR023
+L GND #PWR025
 U 1 1 4F9A6571
 P 2250 5350
-F 0 "#PWR023" H 2250 5350 30  0001 C CNN
+F 0 "#PWR025" H 2250 5350 30  0001 C CNN
 F 1 "GND" H 2250 5280 30  0001 C CNN
 	1    2250 5350
@@
 $EndComp
 $Comp
-L GND #PWR024
+L GND #PWR026
 U 1 1 4F9A6577
 P 2250 5650
-F 0 "#PWR024" H 2250 5650 30  0001 C CNN
+F 0 "#PWR026" H 2250 5650 30  0001 C CNN
 F 1 "GND" H 2250 5580 30  0001 C CNN
 	1    2250 5650
@@
 SCI_GPIO_2
 Text Label 6550 2850 0    60   ~ 0
-SCI_GPIO_1
+SCI_GPIO_0
 Text Label 6550 2750 0    60   ~ 0
 SCI_GPIO_1
@@
 $EndComp
 $Comp
-L SCI_AVDD_5_5V #PWR025
+L SCI_AVDD_5_5V #PWR027
 U 1 1 4F9A6596
 P 1350 3850
-F 0 "#PWR025" H 1350 3950 30  0001 C CNN
+F 0 "#PWR027" H 1350 3950 30  0001 C CNN
 F 1 "SCI_AVDD_5_5V" H 1350 3950 30  0000 C CNN
 	1    1350 3850
@@
 $EndComp
 $Comp
-L AFE/SCI_ANLG_VDD #PWR026
+L AFE/SCI_ANLG_VDD #PWR028
 U 1 1 4F9A65A5
 P 1850 5700
-F 0 "#PWR026" H 1850 5800 30  0001 C CNN
+F 0 "#PWR028" H 1850 5800 30  0001 C CNN
 F 1 "AFE/SCI_ANLG_VDD" H 1850 5800 30  0000 C CNN
 	1    1850 5700
@@
 $EndComp
 $Comp
-L AFE/SCI_ANLG_VSS #PWR027
+L AFE/SCI_ANLG_VSS #PWR029
 U 1 1 4F9A65AB
 P 1850 5950
-F 0 "#PWR027" H 1850 5850 30  0001 C CNN
+F 0 "#PWR029" H 1850 5850 30  0001 C CNN
 F 1 "AFE/SCI_ANLG_VSS" H 1850 5850 30  0000 C CNN
 	1    1850 5950
@@
 SCI_PWR_GOOD
 $Comp
-L AFE/SCI_VREF_VDD #PWR028
+L AFE/SCI_VREF_VDD #PWR030
 U 1 1 4F9A65B2
 P 1850 4650
-F 0 "#PWR028" H 1850 4750 30  0001 C CNN
+F 0 "#PWR030" H 1850 4750 30  0001 C CNN
 F 1 "AFE/SCI_VREF_VDD" H 1850 4750 30  0000 C CNN
 	1    1850 4650
@@
 $EndComp
 $Comp
-L AFE/SCI_VREF_VSS #PWR029
+L AFE/SCI_VREF_VSS #PWR031
 U 1 1 4F9A65B8
 P 1850 4900
-F 0 "#PWR029" H 1850 4800 30  0001 C CNN
+F 0 "#PWR031" H 1850 4800 30  0001 C CNN
 F 1 "AFE/SCI_VREF_VSS" H 1850 4800 30  0000 C CNN
 	1    1850 4900
@@
 AFE/SCI_VREF
 $Comp
-L AFE/SCI_VREF_VSS #PWR030
+L AFE/SCI_VREF_VSS #PWR032
 U 1 1 4F9A65BF
 P 9300 4350
-F 0 "#PWR030" H 9300 4250 30  0001 C CNN
+F 0 "#PWR032" H 9300 4250 30  0001 C CNN
 F 1 "AFE/SCI_VREF_VSS" H 9300 4250 30  0000 C CNN
 	1    9300 4350
@@
 $EndComp
 $Comp
-L AFE/SCI_ANLG_VSS #PWR031
+L AFE/SCI_ANLG_VSS #PWR033
 U 1 1 4F9A65C5
 P 8800 4350
-F 0 "#PWR031" H 8800 4250 30  0001 C CNN
+F 0 "#PWR033" H 8800 4250 30  0001 C CNN
 F 1 "AFE/SCI_ANLG_VSS" H 8800 4250 30  0000 C CNN
 	1    8800 4350
@@
 $EndComp
 $Comp
-L AFE/SCI_ANLG_VDD #PWR032
+L AFE/SCI_ANLG_VDD #PWR034
 U 1 1 4F9A65CB
 P 8800 3200
-F 0 "#PWR032" H 8800 3300 30  0001 C CNN
+F 0 "#PWR034" H 8800 3300 30  0001 C CNN
 F 1 "AFE/SCI_ANLG_VDD" H 8800 3300 30  0000 C CNN
 	1    8800 3200
@@
 $EndComp
 $Comp
-L SCI_AVDD_5_5V #PWR033
+L SCI_AVDD_5_5V #PWR035
 U 1 1 4F9A65D1
 P 8250 3200
-F 0 "#PWR033" H 8250 3300 30  0001 C CNN
+F 0 "#PWR035" H 8250 3300 30  0001 C CNN
 F 1 "SCI_AVDD_5_5V" H 8250 3300 30  0000 C CNN
 	1    8250 3200
@@
 $EndComp
 $Comp
-L GND #PWR034
+L GND #PWR036
 U 1 1 4F9A65D7
 P 9650 4200
-F 0 "#PWR034" H 9650 4200 30  0001 C CNN
+F 0 "#PWR036" H 9650 4200 30  0001 C CNN
 F 1 "GND" H 9650 4130 30  0001 C CNN
 	1    9650 4200
@@
 AFE/SCI_VREF
 $Comp
-L AFE/SCI_VREF_VDD #PWR035
+L AFE/SCI_VREF_VDD #PWR037
 U 1 1 4F9A65DF
 P 9300 3200
-F 0 "#PWR035" H 9300 3300 30  0001 C CNN
+F 0 "#PWR037" H 9300 3300 30  0001 C CNN
 F 1 "AFE/SCI_VREF_VDD" H 9300 3300 30  0000 C CNN
 	1    9300 3200
@@
 $EndComp
 $Comp
-L GND #PWR036
+L GND #PWR038
 U 1 1 4F9A65E5
 P 9650 3350
-F 0 "#PWR036" H 9650 3350 30  0001 C CNN
+F 0 "#PWR038" H 9650 3350 30  0001 C CNN
 F 1 "GND" H 9650 3280 30  0001 C CNN
 	1    9650 3350
@@
 $EndComp
 $Comp
-L GND #PWR037
+L GND #PWR039
 U 1 1 4F9A65F4
 P 5150 6500
-F 0 "#PWR037" H 5150 6500 30  0001 C CNN
+F 0 "#PWR039" H 5150 6500 30  0001 C CNN
 F 1 "GND" H 5150 6430 30  0001 C CNN
 	1    5150 6500
@@
 $EndComp
 $Comp
-L SCI_DVDD_3_3V #PWR038
+L SCI_DVDD_3_3V #PWR040
 U 1 1 4F9A6603
 P 850 4150
-F 0 "#PWR038" H 850 4250 30  0001 C CNN
+F 0 "#PWR040" H 850 4250 30  0001 C CNN
 F 1 "SCI_DVDD_3_3V" H 850 4250 30  0000 C CNN
 	1    850  4150
@@
 $EndComp
 $Comp
-L SCI_DVDD_3_3V #PWR039
+L SCI_DVDD_3_3V #PWR041
 U 1 1 4F9A6609
 P 8400 4000
-F 0 "#PWR039" H 8400 4100 30  0001 C CNN
+F 0 "#PWR041" H 8400 4100 30  0001 C CNN
 F 1 "SCI_DVDD_3_3V" H 8400 4100 30  0000 C CNN
 	1    8400 4000
@@
 	7100 2750 6500 2750
 Wire Wire Line
-	7100 2850 6500 2850
+	7250 2850 6500 2850
 Wire Wire Line
 	7100 2650 6500 2650
@@
 	5700 3500 5700 3250
 Wire Wire Line
-	5050 3500 5700 3500
+	5000 3500 5700 3500
 Wire Wire Line
 	5550 2850 5750 2850
@@
 Connection ~ 850  4250
 Connection ~ 850  4250
+Text HLabel 7250 2850 2    60   Output ~ 0
+SCI_GPIO_0
 $EndSCHEMATC

Commit message: Fixed component properties to make the BOM look nicer
Parts:
- R3, R4: Description RES THICK FILM 0.10 OHM 0.25W ±1% 0805 -> RES THICK FILM 0.10 OHM 0.25W 1% 0805
Changed lines of the file:
@@
-EESchema Schematic File Version 2  date Fri 27 Apr 2012 11:11:24 AM EDT
+EESchema Schematic File Version 2  date Fri 27 Apr 2012 12:40:07 PM EDT
 LIBS:custom_transistors
 LIBS:TI_custom
@@
 F 4 "Yageo" H 1700 3950 60  0001 C CNN "Manufacturer"
 F 5 "PT0805FR-7W0R1L" H 1700 3950 60  0001 C CNN "Part Number"
-F 6 "RES THICK FILM 0.10 OHM 0.25W ±1% 0805" H 1700 3950 60  0001 C CNN "Description"
+F 6 "RES THICK FILM 0.10 OHM 0.25W 1% 0805" H 1700 3950 60  0001 C CNN "Description"
 	1    1700 3950
 	1    0    0    -1
@@
 F 4 "Yageo" H 1200 4250 60  0001 C CNN "Manufacturer"
 F 5 "PT0805FR-7W0R1L" H 1200 4250 60  0001 C CNN "Part Number"
-F 6 "RES THICK FILM 0.10 OHM 0.25W ±1% 0805" H 1200 4250 60  0001 C CNN "Description"
+F 6 "RES THICK FILM 0.10 OHM 0.25W 1% 0805" H 1200 4250 60  0001 C CNN "Description"
 	1    1200 4250
 	1    0    0    -1

Commit message: Fixed more component properties to make the BOM look nice
Parts:
- R3, R4: footprint SM0805 -> 0805
Changed lines of the file:
@@
-EESchema Schematic File Version 2  date Fri 27 Apr 2012 12:40:07 PM EDT
+EESchema Schematic File Version 2  date Fri 27 Apr 2012 12:41:37 PM EDT
 LIBS:custom_transistors
 LIBS:TI_custom
@@
 F 0 "R4" H 1700 4050 50  0000 C CNN
 F 1 "0.10" H 1700 3850 50  0000 C CNN
-F 2 "SM0805" H 1700 3950 60  0001 C CNN
+F 2 "0805" H 1700 3950 60  0001 C CNN
 F 4 "Yageo" H 1700 3950 60  0001 C CNN "Manufacturer"
 F 5 "PT0805FR-7W0R1L" H 1700 3950 60  0001 C CNN "Part Number"
@@
 F 0 "R3" H 1200 4350 50  0000 C CNN
 F 1 "0.10" H 1200 4150 50  0000 C CNN
-F 2 "SM0805" H 1200 4250 60  0001 C CNN
+F 2 "0805" H 1200 4250 60  0001 C CNN
 F 4 "Yageo" H 1200 4250 60  0001 C CNN "Manufacturer"
 F 5 "PT0805FR-7W0R1L" H 1200 4250 60  0001 C CNN "Part Number"

Commit message: Enlarged the text on all of the power rails to make them easier to see when plotted
Connections:
- wire segments 162 -> 172
Other:
- moved on the sheet: P4, P5, R3, R4

Commit message: Re-annotated for added parts.
Connections:
- wire segments 172 -> 162
Changed lines of the file:
@@
-EESchema Schematic File Version 2  date Fri 27 Apr 2012 02:46:40 PM EDT
+EESchema Schematic File Version 2  date Wed 02 May 2012 02:37:03 AM EDT
 LIBS:custom_transistors
 LIBS:TI_custom
@@
 Sheet 5 9
 Title "SCI-BREADBRD-MVK"
-Date "27 apr 2012"
+Date "2 may 2012"
 Rev "A"
 Comp "The Ohio State University"
@@
 $EndComp
 $Comp
-L GND #PWR28
+L GND #PWR016
 U 1 1 4F9A653B
 P 2500 6500
-F 0 "#PWR28" H 2500 6500 30  0001 C CNN
+F 0 "#PWR016" H 2500 6500 30  0001 C CNN
 F 1 "GND" H 2500 6430 30  0001 C CNN
 	1    2500 6500
@@
 $EndComp
 $Comp
-L GND #PWR30
+L GND #PWR017
 U 1 1 4F9A6541
 P 5400 2950
-F 0 "#PWR30" H 5400 2950 30  0001 C CNN
+F 0 "#PWR017" H 5400 2950 30  0001 C CNN
 F 1 "GND" H 5400 2880 30  0001 C CNN
 	1    5400 2950
@@
 $EndComp
 $Comp
-L GND #PWR29
+L GND #PWR018
 U 1 1 4F9A6547
 P 5400 2200
-F 0 "#PWR29" H 5400 2200 30  0001 C CNN
+F 0 "#PWR018" H 5400 2200 30  0001 C CNN
 F 1 "GND" H 5400 2130 30  0001 C CNN
 	1    5400 2200
@@
 $EndComp
 $Comp
-L GND #PWR20
+L GND #PWR019
 U 1 1 4F9A654D
 P 2500 2200
-F 0 "#PWR20" H 2500 2200 30  0001 C CNN
+F 0 "#PWR019" H 2500 2200 30  0001 C CNN
 F 1 "GND" H 2500 2130 30  0001 C CNN
 	1    2500 2200
@@
 $EndComp
 $Comp
-L GND #PWR21
+L GND #PWR020
 U 1 1 4F9A6553
 P 2500 2950
-F 0 "#PWR21" H 2500 2950 30  0001 C CNN
+F 0 "#PWR020" H 2500 2950 30  0001 C CNN
 F 1 "GND" H 2500 2880 30  0001 C CNN
 	1    2500 2950
@@
 $EndComp
 $Comp
-L GND #PWR22
+L GND #PWR021
 U 1 1 4F9A6559
 P 2500 3400
-F 0 "#PWR22" H 2500 3400 30  0001 C CNN
+F 0 "#PWR021" H 2500 3400 30  0001 C CNN
 F 1 "GND" H 2500 3330 30  0001 C CNN
 	1    2500 3400
@@
 $EndComp
 $Comp
-L GND #PWR23
+L GND #PWR022
 U 1 1 4F9A655F
 P 2500 3850
-F 0 "#PWR23" H 2500 3850 30  0001 C CNN
+F 0 "#PWR022" H 2500 3850 30  0001 C CNN
 F 1 "GND" H 2500 3780 30  0001 C CNN
 	1    2500 3850
@@
 $EndComp
 $Comp
-L GND #PWR24
+L GND #PWR023
 U 1 1 4F9A6565
 P 2500 4600
-F 0 "#PWR24" H 2500 4600 30  0001 C CNN
+F 0 "#PWR023" H 2500 4600 30  0001 C CNN
 F 1 "GND" H 2500 4530 30  0001 C CNN
 	1    2500 4600
@@
 $EndComp
 $Comp
-L GND #PWR25
+L GND #PWR024
 U 1 1 4F9A656B
 P 2500 5050
-F 0 "#PWR25" H 2500 5050 30  0001 C CNN
+F 0 "#PWR024" H 2500 5050 30  0001 C CNN
 F 1 "GND" H 2500 4980 30  0001 C CNN
 	1    2500 5050
@@
 $EndComp
 $Comp
-L GND #PWR26
+L GND #PWR025
 U 1 1 4F9A6571
 P 2500 5350
-F 0 "#PWR26" H 2500 5350 30  0001 C CNN
+F 0 "#PWR025" H 2500 5350 30  0001 C CNN
 F 1 "GND" H 2500 5280 30  0001 C CNN
 	1    2500 5350
@@
 $EndComp
 $Comp
-L GND #PWR27
+L GND #PWR026
 U 1 1 4F9A6577
 P 2500 5650
-F 0 "#PWR27" H 2500 5650 30  0001 C CNN
+F 0 "#PWR026" H 2500 5650 30  0001 C CNN
 F 1 "GND" H 2500 5580 30  0001 C CNN
 	1    2500 5650
@@
 $EndComp
 $Comp
-L AFE/SCI_ANLG_VDD #PWR18
+L AFE/SCI_ANLG_VDD #PWR027
 U 1 1 4F9A65A5
 P 2100 5700
-F 0 "#PWR18" H 2100 5800 30  0001 C CNN
+F 0 "#PWR027" H 2100 5800 30  0001 C CNN
 F 1 "AFE/SCI_ANLG_VDD" H 2100 5800 30  0000 C CNN
 	1    2100 5700
@@
 $EndComp
 $Comp
-L AFE/SCI_ANLG_VSS #PWR19
+L AFE/SCI_ANLG_VSS #PWR028
 U 1 1 4F9A65AB
 P 2100 5950
-F 0 "#PWR19" H 2100 5850 30  0001 C CNN
+F 0 "#PWR028" H 2100 5850 30  0001 C CNN
 F 1 "AFE/SCI_ANLG_VSS" H 2100 5850 30  0000 C CNN
 	1    2100 5950
@@
 SCI_PWR_GOOD
 $Comp
-L AFE/SCI_VREF_VDD #PWR16
+L AFE/SCI_VREF_VDD #PWR029
 U 1 1 4F9A65B2
 P 2100 4650
-F 0 "#PWR16" H 2100 4750 30  0001 C CNN
+F 0 "#PWR029" H 2100 4750 30  0001 C CNN
 F 1 "AFE/SCI_VREF_VDD" H 2100 4750 30  0000 C CNN
 	1    2100 4650
@@
 $EndComp
 $Comp
-L AFE/SCI_VREF_VSS #PWR17
+L AFE/SCI_VREF_VSS #PWR030
 U 1 1 4F9A65B8
 P 2100 4900
-F 0 "#PWR17" H 2100 4800 30  0001 C CNN
+F 0 "#PWR030" H 2100 4800 30  0001 C CNN
 F 1 "AFE/SCI_VREF_VSS" H 2100 4800 30  0000 C CNN
 	1    2100 4900
@@
 AFE/SCI_VREF
 $Comp
-L GND #PWR39
+L GND #PWR031
 U 1 1 4F9A65D7
 P 9900 4200
-F 0 "#PWR39" H 9900 4200 30  0001 C CNN
+F 0 "#PWR031" H 9900 4200 30  0001 C CNN
 F 1 "GND" H 9900 4130 30  0001 C CNN
 	1    9900 4200
@@
 AFE/SCI_VREF
 $Comp
-L GND #PWR38
+L GND #PWR032
 U 1 1 4F9A65E5
 P 9900 3350
-F 0 "#PWR38" H 9900 3350 30  0001 C CNN
+F 0 "#PWR032" H 9900 3350 30  0001 C CNN
 F 1 "GND" H 9900 3280 30  0001 C CNN
 	1    9900 3350
@@
 $EndComp
 $Comp
-L GND #PWR31
+L GND #PWR033
 U 1 1 4F9A65F4
 P 5400 6500
-F 0 "#PWR31" H 5400 6500 30  0001 C CNN
+F 0 "#PWR033" H 5400 6500 30  0001 C CNN
 F 1 "GND" H 5400 6430 30  0001 C CNN
 	1    5400 6500
@@
 SCI_GPIO_0
 $Comp
-L SCI_AVDD_5_5V #PWR?
+L SCI_AVDD_5_5V #PWR034
 U 1 1 4F9AE708
 P 8500 3200
-F 0 "#PWR?" H 8500 3300 30  0001 C CNN
+F 0 "#PWR034" H 8500 3300 30  0001 C CNN
 F 1 "SCI_AVDD_5_5V" H 8500 3300 60  0000 C CNN
 	1    8500 3200
@@
 $EndComp
 $Comp
-L AFE/SCI_ANLG_VDD #PWR?
+L AFE/SCI_ANLG_VDD #PWR035
 U 1 1 4F9AE777
 P 9050 2850
-F 0 "#PWR?" H 9050 2950 30  0001 C CNN
+F 0 "#PWR035" H 9050 2950 30  0001 C CNN
 F 1 "AFE/SCI_ANLG_VDD" H 9050 2950 60  0000 C CNN
 	1    9050 2850
@@
 $EndComp
 $Comp
-L AFE/SCI_VREF_VDD #PWR?
+L AFE/SCI_VREF_VDD #PWR036
 U 1 1 4F9AE7DC
 P 9550 3100
-F 0 "#PWR?" H 9550 3200 30  0001 C CNN
+F 0 "#PWR036" H 9550 3200 30  0001 C CNN
 F 1 "AFE/SCI_VREF_VDD" H 9550 3200 60  0000 C CNN
 	1    9550 3100
@@
 	1450 3950 1700 3950
 Wire Wire Line
-	1450 3850 1450 3950
-Wire Wire Line
-	1450 3950 1450 4100
+	1450 3850 1450 4100
 Wire Wire Line
 	1450 4100 2650 4100
@@
 	2500 6250 2650 6250
 Wire Wire Line
-	2500 6250 2500 6350
-Wire Wire Line
-	2500 6350 2500 6500
+	2500 6250 2500 6500
 Wire Wire Line
 	2650 6350 2500 6350
@@
 	5400 6250 5250 6250
 Wire Wire Line
-	5400 6250 5400 6350
-Wire Wire Line
-	5400 6350 5400 6500
+	5400 6250 5400 6500
 Wire Wire Line
 	5250 6350 5400 6350
@@
 	8500 3200 8500 3300
 Wire Wire Line
-	8500 3300 9050 3300
-Wire Wire Line
-	9050 3300 9150 3300
+	8500 3300 9150 3300
 Wire Wire Line
 	8550 4000 8550 4150
 Wire Wire Line
-	8550 4150 9050 4150
-Wire Wire Line
-	9050 4150 9150 4150
+	8550 4150 9150 4150
 Wire Wire Line
 	9050 2850 9050 3250
 Wire Wire Line
-	9050 3250 9250 3250
-Wire Wire Line
-	9250 3250 9350 3250
+	9050 3250 9350 3250
 Wire Wire Line
 	9250 3250 9250 3350
 Wire Wire Line
-	9550 4100 9550 4150
-Wire Wire Line
-	9550 4150 9550 4550
+	9550 4100 9550 4550
 Wire Wire Line
 	9250 4100 9250 4200
@@
 Connection ~ 9250 3250
 Wire Wire Line
-	9550 3100 9550 3250
-Wire Wire Line
-	9550 3250 9550 3350
+	9550 3100 9550 3350
 Wire Wire Line
 	9550 3250 9450 3250
@@
 Connection ~ 9550 3250
 Wire Wire Line
-	8800 4200 9250 4200
-Wire Wire Line
-	9250 4200 9350 4200
+	8800 4200 9350 4200
 Wire Wire Line
 	9350 4200 9350 4100
@@
 	9650 4100 9650 4400
 Wire Wire Line
-	950  4150 950  4250
-Wire Wire Line
-	950  4250 950  4400
+	950  4150 950  4400
 Connection ~ 950  4250
 Connection ~ 950  4250
 $Comp
-L SCI_DVDD_3_3V #PWR?
+L SCI_DVDD_3_3V #PWR037
 U 1 1 4F9AE9BB
 P 8550 4000
-F 0 "#PWR?" H 8550 4100 30  0001 C CNN
+F 0 "#PWR037" H 8550 4100 30  0001 C CNN
 F 1 "SCI_DVDD_3_3V" H 8550 4150 60  0000 C CNN
 	1    8550 4000
@@
 $EndComp
 $Comp
-L AFE/SCI_ANLG_VSS #PWR?
+L AFE/SCI_ANLG_VSS #PWR038
 U 1 1 4F9AEA34
 P 8800 4350
-F 0 "#PWR?" H 8800 4250 30  0001 C CNN
+F 0 "#PWR038" H 8800 4250 30  0001 C CNN
 F 1 "AFE/SCI_ANLG_VSS" H 8800 4200 60  0000 C CNN
 	1    8800 4350
@@
 $EndComp
 $Comp
-L AFE/SCI_VREF_VSS #PWR?
+L AFE/SCI_VREF_VSS #PWR039
 U 1 1 4F9AEAA3
 P 9550 4550
-F 0 "#PWR?" H 9550 4450 30  0001 C CNN
+F 0 "#PWR039" H 9550 4450 30  0001 C CNN
 F 1 "AFE/SCI_VREF_VSS" H 9550 4400 60  0000 C CNN
 	1    9550 4550
@@
 $EndComp
 $Comp
-L SCI_AVDD_5_5V #PWR?
+L SCI_AVDD_5_5V #PWR040
 U 1 1 4F9AEAB2
 P 1450 3850
-F 0 "#PWR?" H 1450 3950 30  0001 C CNN
+F 0 "#PWR040" H 1450 3950 30  0001 C CNN
 F 1 "SCI_AVDD_5_5V" H 1450 3950 60  0000 C CNN
 	1    1450 3850
@@
 $EndComp
 $Comp
-L SCI_DVDD_3_3V #PWR?
+L SCI_DVDD_3_3V #PWR041
 U 1 1 4F9AEAC1
 P 950 4150
-F 0 "#PWR?" H 950 4250 30  0001 C CNN
+F 0 "#PWR041" H 950 4250 30  0001 C CNN
 F 1 "SCI_DVDD_3_3V" H 950 4300 60  0000 C CNN
 	1    950  4150

Commit message: Added some bypass caps. Rearranged pins on connectors to make layout easier.
Connections:
- wire segments 162 -> 172
