File: SCI-BREADBRD_sci_conn.sch (KiCad schematic (older format))
At the start: 6 parts, among them P4 MARK_SCI_CONN, P5 CONN_16, P6 CONN_8X2, P7 CONN_8X2

Commit message: More layout progress
Changed lines of the file:
@@
-EESchema Schematic File Version 2  date Wed 02 May 2012 11:48:38 PM EDT
+EESchema Schematic File Version 2  date Fri 04 May 2012 05:15:56 PM EDT
 LIBS:custom_transistors
 LIBS:TI_custom
@@
 Sheet 5 9
 Title "SCI-BREADBRD-MVK"
-Date "3 may 2012"
+Date "4 may 2012"
 Rev "A"
 Comp "The Ohio State University"
@@
 Text Label 1700 5150 0    60   ~ 0
 AFE/SCI_VREF
-Text Label 9250 5750 0    60   ~ 0
+Text Label 8900 6000 0    60   ~ 0
 SCI_PWR_GOOD
-Text Label 9000 4600 0    60   ~ 0
+Text Label 8950 4350 0    60   ~ 0
 AFE/SCI_VREF
 $Comp
-L GND #PWR032
+L GND #PWR031
 U 1 1 4F9A65E5
 P 9450 4900
-F 0 "#PWR032" H 9450 4900 30  0001 C CNN
+F 0 "#PWR031" H 9450 4900 30  0001 C CNN
 F 1 "GND" H 9450 4830 30  0001 C CNN
 	1    9450 4900
@@
 $EndComp
 $Comp
-L GND #PWR033
+L GND #PWR032
 U 1 1 4F9A65F4
 P 5400 6500
-F 0 "#PWR033" H 5400 6500 30  0001 C CNN
+F 0 "#PWR032" H 5400 6500 30  0001 C CNN
 F 1 "GND" H 5400 6430 30  0001 C CNN
 	1    5400 6500
@@
 SCI_GPIO_0
 $Comp
-L SCI_AVDD_5_5V #PWR034
+L SCI_AVDD_5_5V #PWR033
 U 1 1 4F9AE708
 P 7650 4650
-F 0 "#PWR034" H 7650 4750 30  0001 C CNN
+F 0 "#PWR033" H 7650 4750 30  0001 C CNN
 F 1 "SCI_AVDD_5_5V" H 7650 4750 60  0000 C CNN
 	1    7650 4650
@@
 $EndComp
 $Comp
-L AFE/SCI_ANLG_VDD #PWR035
+L AFE/SCI_ANLG_VDD #PWR034
 U 1 1 4F9AE777
-P 8600 4300
-F 0 "#PWR035" H 8600 4400 30  0001 C CNN
-F 1 "AFE/SCI_ANLG_VDD" H 8600 4450 60  0000 C CNN
-	1    8600 4300
-	1    0    0    -1
-$EndComp
-$Comp
-L AFE/SCI_VREF_VDD #PWR036
+P 10150 3850
+F 0 "#PWR034" H 10150 3950 30  0001 C CNN
+F 1 "AFE/SCI_ANLG_VDD" H 10150 4000 60  0000 C CNN
+	1    10150 3850
+	1    0    0    -1
+$EndComp
+$Comp
+L AFE/SCI_VREF_VDD #PWR035
 U 1 1 4F9AE7DC
-P 9650 3950
-F 0 "#PWR036" H 9650 4050 30  0001 C CNN
-F 1 "AFE/SCI_VREF_VDD" H 9650 4050 60  0000 C CNN
-	1    9650 3950
-	1    0    0    -1
-$EndComp
-$Comp
-L SCI_DVDD_3_3V #PWR037
+P 8600 4250
+F 0 "#PWR035" H 8600 4350 30  0001 C CNN
+F 1 "AFE/SCI_VREF_VDD" H 8600 4350 60  0000 C CNN
+	1    8600 4250
+	1    0    0    -1
+$EndComp
+$Comp
+L SCI_DVDD_3_3V #PWR036
 U 1 1 4F9AE9BB
 P 8100 4500
-F 0 "#PWR037" H 8100 4600 30  0001 C CNN
+F 0 "#PWR036" H 8100 4600 30  0001 C CNN
 F 1 "SCI_DVDD_3_3V" H 8100 4650 60  0000 C CNN
 	1    8100 4500
@@
 $EndComp
 $Comp
-L AFE/SCI_VREF_VSS #PWR039
+L AFE/SCI_VREF_VSS #PWR037
 U 1 1 4F9AEAA3
-P 10150 3850
-F 0 "#PWR039" H 10150 3750 30  0001 C CNN
-F 1 "AFE/SCI_VREF_VSS" H 10150 3700 60  0000 C CNN
-	1    10150 3850
+P 9100 4150
+F 0 "#PWR037" H 9100 4050 30  0001 C CNN
+F 1 "AFE/SCI_VREF_VSS" H 9100 4000 60  0000 C CNN
+	1    9100 4150
 	-1   0    0    1
 $EndComp
 $Comp
-L SCI_AVDD_5_5V #PWR040
+L SCI_AVDD_5_5V #PWR038
 U 1 1 4F9AEAB2
 P 1450 3850
-F 0 "#PWR040" H 1450 3950 30  0001 C CNN
+F 0 "#PWR038" H 1450 3950 30  0001 C CNN
 F 1 "SCI_AVDD_5_5V" H 1450 3950 60  0000 C CNN
 	1    1450 3850
@@
 $EndComp
 $Comp
-L SCI_DVDD_3_3V #PWR041
+L SCI_DVDD_3_3V #PWR039
 U 1 1 4F9AEAC1
 P 950 4150
-F 0 "#PWR041" H 950 4250 30  0001 C CNN
+F 0 "#PWR039" H 950 4250 30  0001 C CNN
 F 1 "SCI_DVDD_3_3V" H 950 4300 60  0000 C CNN
 	1    950  4150
@@
 $EndComp
 $Comp
-L AFE/SCI_ANLG_VSS #PWR?
+L AFE/SCI_ANLG_VSS #PWR040
 U 1 1 4FA203DC
-P 9100 4150
-F 0 "#PWR?" H 9100 4050 30  0001 C CNN
-F 1 "AFE/SCI_ANLG_VSS" H 9100 4000 60  0000 C CNN
-	1    9100 4150
+P 10700 4100
+F 0 "#PWR040" H 10700 4000 30  0001 C CNN
+F 1 "AFE/SCI_ANLG_VSS" H 10700 3950 60  0000 C CNN
+	1    10700 4100
 	-1   0    0    1
 $EndComp
 $Comp
-L SCI_AVDD_5_5V #PWR?
+L SCI_AVDD_5_5V #PWR041
 U 1 1 4FA208CF
 P 7650 5700
-F 0 "#PWR?" H 7650 5800 30  0001 C CNN
+F 0 "#PWR041" H 7650 5800 30  0001 C CNN
 F 1 "SCI_AVDD_5_5V" H 7650 5800 60  0000 C CNN
 	1    7650 5700
@@
 $EndComp
 $Comp
-L AFE/SCI_ANLG_VDD #PWR?
+L AFE/SCI_ANLG_VDD #PWR042
 U 1 1 4FA208D5
-P 8600 6050
-F 0 "#PWR?" H 8600 6150 30  0001 C CNN
-F 1 "AFE/SCI_ANLG_VDD" H 8600 6200 60  0000 C CNN
-	1    8600 6050
+P 9850 6500
+F 0 "#PWR042" H 9850 6600 30  0001 C CNN
+F 1 "AFE/SCI_ANLG_VDD" H 9850 6650 60  0000 C CNN
+	1    9850 6500
 	1    0    0    1
 $EndComp
 $Comp
-L AFE/SCI_VREF_VDD #PWR?
+L AFE/SCI_VREF_VDD #PWR043
 U 1 1 4FA208DB
-P 9650 6400
-F 0 "#PWR?" H 9650 6500 30  0001 C CNN
-F 1 "AFE/SCI_VREF_VDD" H 9650 6500 60  0000 C CNN
-	1    9650 6400
+P 8600 6100
+F 0 "#PWR043" H 8600 6200 30  0001 C CNN
+F 1 "AFE/SCI_VREF_VDD" H 8600 6200 60  0000 C CNN
+	1    8600 6100
 	1    0    0    1
 $EndComp
 $Comp
-L SCI_DVDD_3_3V #PWR?
+L SCI_DVDD_3_3V #PWR044
 U 1 1 4FA208E1
 P 8100 5850
-F 0 "#PWR?" H 8100 5950 30  0001 C CNN
+F 0 "#PWR044" H 8100 5950 30  0001 C CNN
 F 1 "SCI_DVDD_3_3V" H 8100 6000 60  0000 C CNN
 	1    8100 5850
@@
 $EndComp
 $Comp
-L AFE/SCI_VREF_VSS #PWR?
+L AFE/SCI_VREF_VSS #PWR045
 U 1 1 4FA208E7
-P 10150 6500
-F 0 "#PWR?" H 10150 6400 30  0001 C CNN
-F 1 "AFE/SCI_VREF_VSS" H 10150 6350 60  0000 C CNN
-	1    10150 6500
-	-1   0    0    -1
-$EndComp
-$Comp
-L AFE/SCI_ANLG_VSS #PWR?
+P 9100 6200
+F 0 "#PWR045" H 9100 6100 30  0001 C CNN
+F 1 "AFE/SCI_VREF_VSS" H 9100 6050 60  0000 C CNN
+	1    9100 6200
+	-1   0    0    -1
+$EndComp
+$Comp
+L AFE/SCI_ANLG_VSS #PWR046
 U 1 1 4FA208ED
-P 9100 6200
-F 0 "#PWR?" H 9100 6100 30  0001 C CNN
-F 1 "AFE/SCI_ANLG_VSS" H 9100 6050 60  0000 C CNN
-	1    9100 6200
-	-1   0    0    -1
-$EndComp
-$Comp
-L GND #PWR?
+P 10350 6200
+F 0 "#PWR046" H 10350 6100 30  0001 C CNN
+F 1 "AFE/SCI_ANLG_VSS" H 10350 6050 60  0000 C CNN
+	1    10350 6200
+	-1   0    0    -1
+$EndComp
+$Comp
+L GND #PWR047
 U 1 1 4FA20908
-P 10300 5750
-F 0 "#PWR?" H 10300 5750 30  0001 C CNN
-F 1 "GND" H 10300 5680 30  0001 C CNN
-	1    10300 5750
+P 10600 5750
+F 0 "#PWR047" H 10600 5750 30  0001 C CNN
+F 1 "GND" H 10600 5680 30  0001 C CNN
+	1    10600 5750
 	-1   0    0    -1
 $EndComp
@@
 	2650 5150 1700 5150
 Wire Wire Line
-	9000 5750 9950 5750
-Wire Wire Line
 	7650 4650 7650 4750
 Wire Wire Line
 	8100 4500 8100 4700
 Wire Wire Line
-	8600 4300 8600 4800
+	8600 4250 8600 4800
 Wire Wire Line
 	950  4150 950  4400
@@
 	8700 4250 8700 4800
 Wire Wire Line
-	9650 3950 9650 4350
-Wire Wire Line
-	9650 4350 8800 4350
+	8800 4350 9650 4350
 Wire Wire Line
 	8800 4350 8800 4800
@@
 	9000 4800 9000 4600
 Wire Wire Line
-	9000 4600 9550 4600
+	9000 4600 10700 4600
 Wire Wire Line
 	9100 4800 9100 4700
@@
 	8100 5850 8100 5650
 Wire Wire Line
-	8600 6050 8600 5550
+	8600 6100 8600 5550
 Wire Wire Line
 	7650 5600 8400 5600
@@
 	8700 6100 8700 5550
 Wire Wire Line
-	9650 6400 9650 6000
-Wire Wire Line
-	9650 6000 8800 6000
+	8800 6000 9650 6000
 Wire Wire Line
 	8800 6000 8800 5550
 Wire Wire Line
-	10150 6500 10150 5900
-Wire Wire Line
-	10150 5900 8900 5900
+	9850 6500 9850 5900
+Wire Wire Line
+	9850 5900 8900 5900
 Wire Wire Line
 	8900 5900 8900 5550
@@
 	9100 5550 9100 5650
 Wire Wire Line
-	9100 5650 10300 5650
-Wire Wire Line
-	10300 5650 10300 5750
+	9100 5650 10600 5650
+Wire Wire Line
+	10600 5650 10600 5750
+Wire Wire Line
+	10700 4600 10700 4100
+Wire Wire Line
+	9000 5750 10350 5750
+Wire Wire Line
+	10350 5750 10350 6200
 $EndSCHEMATC
