File: SCI-BREADBRD_sci_conn.sch (KiCad schematic (older format))
At the start: 6 parts, among them P4 MARK_SCI_CONN, P5 CONN_16, P6 CONN_8X2, P7 CONN_8X2

Commit message: Finished initial PCB layout
Changed lines of the file:
@@
-EESchema Schematic File Version 2  date Fri 04 May 2012 05:15:56 PM EDT
+EESchema Schematic File Version 2  date Tue 08 May 2012 11:34:32 AM EDT
 LIBS:custom_transistors
 LIBS:TI_custom
@@
 Sheet 5 9
 Title "SCI-BREADBRD-MVK"
-Date "4 may 2012"
+Date "7 may 2012"
 Rev "A"
 Comp "The Ohio State University"
@@
 L GND #PWR018
 U 1 1 4F9A6547
-P 5400 2200
-F 0 "#PWR018" H 5400 2200 30  0001 C CNN
-F 1 "GND" H 5400 2130 30  0001 C CNN
-	1    5400 2200
+P 6150 2200
+F 0 "#PWR018" H 6150 2200 30  0001 C CNN
+F 1 "GND" H 6150 2130 30  0001 C CNN
+	1    6150 2200
 	1    0    0    -1
 $EndComp
@@
 	5250 2900 5400 2900
 Wire Wire Line
-	5400 2150 5400 2200
-Wire Wire Line
-	5250 2150 5400 2150
+	6150 2150 6150 2200
+Wire Wire Line
+	5250 2150 6150 2150
 Connection ~ 2500 6350
 Wire Wire Line
