File: SCI-BREADBRD_vref.sch (KiCad schematic (older format))
At the start: 17 parts

Commit message: Fixed the footprint properties of various parts throughout the schematic to make sure they are all point to valid footprints.
Added SCI-BREADBRD.cmp to specify which footprints should be used for
each part.

Added netlists to the .gitignore as those can be generated easily in
eeschema.
Parts:
- removed U?: OPA454AIDDA, symbol OPA454AIDDA
- added U8: OPA454AIDDA, SOP_8_PowerPad_DDA, symbol OPA454AIDDA
- C17, C18, C19, C20: renamed from C?; footprint SM0402 -> 0402
- P12: renamed from P?; footprint PIN_ARRAY_2x1 -> PIN_ARRAY_2X1
- R22, R23, R24, R25: renamed from R?; footprint SM1210 -> 1210
- R26, R27, R28, R29: renamed from R?; footprint SM0402 -> 0402
- U9: renamed from U?; footprint (none) -> SOP_8_PowerPad_DDA; Description (none) -> IC OPAMP GP 2.5MHZ SGL 8SOIC; Manufacturer (none) -> Texas Instruments; Part Number (none) -> OPA454AIDDA
- gave numbers to parts that had none: 2
Changed lines of the file:
@@
-EESchema Schematic File Version 2  date Fri 27 Apr 2012 04:22:34 AM EDT
+EESchema Schematic File Version 2  date Fri 27 Apr 2012 08:55:37 AM EDT
 LIBS:custom_transistors
 LIBS:TI_custom
@@
 $EndDescr
 $Comp
-L OPA454AIDDA U?
-U 1 1 4F8DFC19
-P 5650 5350
-F 0 "U?" H 5650 5950 60  0000 C CNN
-F 1 "OPA454AIDDA" H 5650 4700 60  0000 C CNN
-	1    5650 5350
-	1    0    0    -1
-$EndComp
-$Comp
-L AFE/SCI_ANLG_VDD #PWR?
+L AFE/SCI_ANLG_VDD #PWR075
 U 1 1 4F8F9D48
 P 4600 4350
-F 0 "#PWR?" H 4600 4450 30  0001 C CNN
+F 0 "#PWR075" H 4600 4450 30  0001 C CNN
 F 1 "AFE/SCI_ANLG_VDD" H 4600 4450 30  0000 C CNN
 	1    4600 4350
@@
 $EndComp
 $Comp
-L AFE/SCI_ANLG_VSS #PWR?
+L AFE/SCI_ANLG_VSS #PWR076
 U 1 1 4F8F9D57
 P 4650 6100
-F 0 "#PWR?" H 4650 6000 30  0001 C CNN
+F 0 "#PWR076" H 4650 6000 30  0001 C CNN
 F 1 "AFE/SCI_ANLG_VSS" H 4650 6000 30  0000 C CNN
 	1    4650 6100
@@
 $EndComp
 $Comp
-L R_US R?
+L R_US R22
 U 1 1 4F8F9D7B
 P 4150 5150
-F 0 "R?" V 4150 5250 50  0000 C CNN
+F 0 "R22" V 4150 5250 50  0000 C CNN
 F 1 "15K" V 4250 5300 50  0000 C CNN
-F 2 "SM1210" H 4150 5150 60  0001 C CNN
+F 2 "1210" H 4150 5150 60  0001 C CNN
 F 4 "Panasonic - ECG" H 4150 5150 60  0001 C CNN "Manufacturer"
 F 5 "ERA-14EB153U" H 4150 5150 60  0001 C CNN "Part Number"
@@
 $EndComp
 $Comp
-L R_US R?
+L R_US R23
 U 1 1 4F8FA0BA
 P 4150 5750
-F 0 "R?" V 4150 5850 50  0000 C CNN
+F 0 "R23" V 4150 5850 50  0000 C CNN
 F 1 "15K" V 4250 5900 50  0000 C CNN
-F 2 "SM1210" H 4150 5750 60  0001 C CNN
+F 2 "1210" H 4150 5750 60  0001 C CNN
 F 4 "Panasonic - ECG" H 4150 5750 60  0001 C CNN "Manufacturer"
 F 5 "ERA-14EB153U" H 4150 5750 60  0001 C CNN "Part Number"
@@
 $EndComp
 $Comp
-L GND #PWR?
+L GND #PWR077
 U 1 1 4F8FA231
 P 6400 5950
-F 0 "#PWR?" H 6400 5950 30  0001 C CNN
+F 0 "#PWR077" H 6400 5950 30  0001 C CNN
 F 1 "GND" H 6400 5880 30  0001 C CNN
 	1    6400 5950
@@
 $EndComp
 $Comp
-L TST P?
+L TST P10
 U 1 1 4F8FA275
 P 7050 4950
-F 0 "P?" H 7050 5250 40  0000 C CNN
+F 0 "P10" H 7050 5250 40  0000 C CNN
 F 1 "SF_ANLG" H 7050 5200 30  0000 C CNN
 F 2 "TESTVIA_p30mil_h20mil" H 7050 4950 60  0001 C CNN
@@
 $EndComp
 $Comp
-L R_US R?
+L R_US R26
 U 1 1 4F8FA2FF
 P 6400 4600
-F 0 "R?" V 6400 4700 50  0000 C CNN
+F 0 "R26" V 6400 4700 50  0000 C CNN
 F 1 "10K" V 6500 4750 50  0000 C CNN
-F 2 "SM0402" H 6400 4600 60  0001 C CNN
+F 2 "0402" H 6400 4600 60  0001 C CNN
 F 4 "Panasonic - ECG" H 6400 4600 60  0001 C CNN "Manufacturer"
 F 5 "ERJ-2GEJ103X" H 6400 4600 60  0001 C CNN "Part Number"
@@
 $EndComp
 $Comp
-L OPA454AIDDA U?
+L OPA454AIDDA U9
 U 1 1 4F8FA888
 P 5700 2650
-F 0 "U?" H 5700 3250 60  0000 C CNN
+F 0 "U9" H 5700 3250 60  0000 C CNN
 F 1 "OPA454AIDDA" H 5700 2000 60  0000 C CNN
+F 2 "SOP_8_PowerPad_DDA" H 5700 2650 60  0001 C CNN
+F 4 "Texas Instruments" H 5700 2650 60  0001 C CNN "Manufacturer"
+F 5 "OPA454AIDDA" H 5700 2650 60  0001 C CNN "Part Number"
+F 6 "IC OPAMP GP 2.5MHZ SGL 8SOIC" H 5700 2650 60  0001 C CNN "Description"
 	1    5700 2650
 	1    0    0    -1
 $EndComp
 $Comp
-L R_US R?
+L R_US R24
 U 1 1 4F8FA89D
 P 4450 2450
-F 0 "R?" V 4450 2550 50  0000 C CNN
+F 0 "R24" V 4450 2550 50  0000 C CNN
 F 1 "15K" V 4550 2600 50  0000 C CNN
-F 2 "SM1210" H 4450 2450 60  0001 C CNN
+F 2 "1210" H 4450 2450 60  0001 C CNN
 F 4 "Panasonic - ECG" H 4450 2450 60  0001 C CNN "Manufacturer"
 F 5 "ERA-14EB153U" H 4450 2450 60  0001 C CNN "Part Number"
@@
 $EndComp
 $Comp
-L R_US R?
+L R_US R25
 U 1 1 4F8FA8A6
 P 4450 3050
-F 0 "R?" V 4450 3150 50  0000 C CNN
+F 0 "R25" V 4450 3150 50  0000 C CNN
 F 1 "15K" V 4550 3200 50  0000 C CNN
-F 2 "SM1210" H 4450 3050 60  0001 C CNN
+F 2 "1210" H 4450 3050 60  0001 C CNN
 F 4 "Panasonic - ECG" H 4450 3050 60  0001 C CNN "Manufacturer"
 F 5 "ERA-14EB153U" H 4450 3050 60  0001 C CNN "Part Number"
@@
 $EndComp
 $Comp
-L GND #PWR?
+L GND #PWR078
 U 1 1 4F8FA8AC
 P 6450 3250
-F 0 "#PWR?" H 6450 3250 30  0001 C CNN
+F 0 "#PWR078" H 6450 3250 30  0001 C CNN
 F 1 "GND" H 6450 3180 30  0001 C CNN
 	1    6450 3250
@@
 $EndComp
 $Comp
-L TST P?
+L TST P11
 U 1 1 4F8FA8B4
 P 7100 2250
-F 0 "P?" H 7100 2550 40  0000 C CNN
+F 0 "P11" H 7100 2550 40  0000 C CNN
 F 1 "SF_MOD" H 7100 2500 30  0000 C CNN
 F 2 "TESTVIA_p30mil_h20mil" H 7100 2250 60  0001 C CNN
@@
 $EndComp
 $Comp
-L R_US R?
+L R_US R27
 U 1 1 4F8FA8C3
 P 6450 1900
-F 0 "R?" V 6450 2000 50  0000 C CNN
+F 0 "R27" V 6450 2000 50  0000 C CNN
 F 1 "10K" V 6550 2050 50  0000 C CNN
-F 2 "SM0402" H 6450 1900 60  0001 C CNN
+F 2 "0402" H 6450 1900 60  0001 C CNN
 F 4 "Panasonic - ECG" H 6450 1900 60  0001 C CNN "Manufacturer"
 F 5 "ERJ-2GEJ103X" H 6450 1900 60  0001 C CNN "Part Number"
@@
 $EndComp
 $Comp
-L MOD_VDD #PWR?
+L MOD_VDD #PWR079
 U 1 1 4F8FA8ED
 P 4650 1650
-F 0 "#PWR?" H 4650 1750 30  0001 C CNN
+F 0 "#PWR079" H 4650 1750 30  0001 C CNN
 F 1 "MOD_VDD" H 4650 1750 30  0000 C CNN
 	1    4650 1650
@@
 $EndComp
 $Comp
-L MOD_VSS #PWR?
+L MOD_VSS #PWR080
 U 1 1 4F8FA8FC
 P 4700 3400
-F 0 "#PWR?" H 4700 3300 30  0001 C CNN
+F 0 "#PWR080" H 4700 3300 30  0001 C CNN
 F 1 "MOD_VSS" H 4700 3300 30  0000 C CNN
 	1    4700 3400
@@
 $EndComp
 $Comp
-L SCI_DVDD_3_3V #PWR?
+L SCI_DVDD_3_3V #PWR081
 U 1 1 4F8FA967
 P 6450 1550
-F 0 "#PWR?" H 6450 1650 30  0001 C CNN
+F 0 "#PWR081" H 6450 1650 30  0001 C CNN
 F 1 "SCI_DVDD_3_3V" H 6450 1650 30  0000 C CNN
 	1    6450 1550
@@
 $EndComp
 $Comp
-L SCI_DVDD_3_3V #PWR?
+L SCI_DVDD_3_3V #PWR082
 U 1 1 4F8FA974
 P 6400 4250
-F 0 "#PWR?" H 6400 4350 30  0001 C CNN
+F 0 "#PWR082" H 6400 4350 30  0001 C CNN
 F 1 "SCI_DVDD_3_3V" H 6400 4350 30  0000 C CNN
 	1    6400 4250
@@
 $EndComp
 $Comp
-L CONN_1X2 P?
+L CONN_1X2 P12
 U 1 1 4F8F7584
 P 8150 3200
-F 0 "P?" V 8150 3200 40  0000 C CNN
+F 0 "P12" V 8150 3200 40  0000 C CNN
 F 1 "CONN_1X2" V 8300 3200 40  0000 C CNN
-F 2 "PIN_ARRAY_2x1" H 8150 3200 60  0001 C CNN
+F 2 "PIN_ARRAY_2X1" H 8150 3200 60  0001 C CNN
 F 4 "Sullins" H 8150 3200 60  0001 C CNN "Manufacturer"
 F 5 "960102-6202-AR" H 8150 3200 60  0001 C CNN "Part Number"
@@
 $EndComp
 $Comp
-L C C?
+L C C19
 U 1 1 4F8F7B49
 P 3950 2400
-F 0 "C?" H 4000 2500 50  0000 L CNN
+F 0 "C19" H 4000 2500 50  0000 L CNN
 F 1 "0.1uF" H 4000 2300 50  0000 L CNN
-F 2 "SM0402" H 3950 2400 60  0001 C CNN
+F 2 "0402" H 3950 2400 60  0001 C CNN
 F 4 "TDK Corporation" H 3950 2400 60  0001 C CNN "Manufacturer"
 F 5 "C1005X6S1H104K" H 3950 2400 60  0001 C CNN "Part Number"
@@
 $EndComp
 $Comp
-L GND #PWR?
+L GND #PWR083
 U 1 1 4F8F7B5C
 P 3950 2700
-F 0 "#PWR?" H 3950 2700 30  0001 C CNN
+F 0 "#PWR083" H 3950 2700 30  0001 C CNN
 F 1 "GND" H 3950 2630 30  0001 C CNN
 	1    3950 2700
@@
 $EndComp
 $Comp
-L C C?
+L C C17
 U 1 1 4F8F8022
 P 3750 4750
-F 0 "C?" H 3800 4850 50  0000 L CNN
+F 0 "C17" H 3800 4850 50  0000 L CNN
 F 1 "0.1uF" H 3800 4650 50  0000 L CNN
-F 2 "SM0402" H 3750 4750 60  0001 C CNN
+F 2 "0402" H 3750 4750 60  0001 C CNN
 F 4 "TDK Corporation" H 3750 4750 60  0001 C CNN "Manufacturer"
 F 5 "C1005X6S1H104K" H 3750 4750 60  0001 C CNN "Part Number"
@@
 $EndComp
 $Comp
-L GND #PWR?
+L GND #PWR084
 U 1 1 4F8F8028
 P 3750 5050
-F 0 "#PWR?" H 3750 5050 30  0001 C CNN
+F 0 "#PWR084" H 3750 5050 30  0001 C CNN
 F 1 "GND" H 3750 4980 30  0001 C CNN
 	1    3750 5050
@@
 $EndComp
 $Comp
-L C C?
+L C C20
 U 1 1 4F8F8397
 P 4100 3650
-F 0 "C?" H 4150 3750 50  0000 L CNN
+F 0 "C20" H 4150 3750 50  0000 L CNN
 F 1 "0.1uF" H 4150 3550 50  0000 L CNN
-F 2 "SM0402" H 4100 3650 60  0001 C CNN
+F 2 "0402" H 4100 3650 60  0001 C CNN
 F 4 "TDK Corporation" H 4100 3650 60  0001 C CNN "Manufacturer"
 F 5 "C1005X6S1H104K" H 4100 3650 60  0001 C CNN "Part Number"
@@
 $EndComp
 $Comp
-L GND #PWR?
+L GND #PWR085
 U 1 1 4F8F839D
 P 4100 3950
-F 0 "#PWR?" H 4100 3950 30  0001 C CNN
+F 0 "#PWR085" H 4100 3950 30  0001 C CNN
 F 1 "GND" H 4100 3880 30  0001 C CNN
 	1    4100 3950
@@
 $EndComp
 $Comp
-L C C?
+L C C18
 U 1 1 4F8F843C
 P 3900 6350
-F 0 "C?" H 3950 6450 50  0000 L CNN
+F 0 "C18" H 3950 6450 50  0000 L CNN
 F 1 "0.1uF" H 3950 6250 50  0000 L CNN
-F 2 "SM0402" H 3900 6350 60  0001 C CNN
+F 2 "0402" H 3900 6350 60  0001 C CNN
 F 4 "TDK Corporation" H 3900 6350 60  0001 C CNN "Manufacturer"
 F 5 "C1005X6S1H104K" H 3900 6350 60  0001 C CNN "Part Number"
@@
 $EndComp
 $Comp
-L GND #PWR?
+L GND #PWR086
 U 1 1 4F8F8442
 P 3900 6650
-F 0 "#PWR?" H 3900 6650 30  0001 C CNN
+F 0 "#PWR086" H 3900 6650 30  0001 C CNN
 F 1 "GND" H 3900 6580 30  0001 C CNN
 	1    3900 6650
@@
 $EndComp
 $Comp
-L R_US R?
+L R_US R29
 U 1 1 4F8F8751
 P 6750 4700
-F 0 "R?" V 6750 4800 50  0000 C CNN
+F 0 "R29" V 6750 4800 50  0000 C CNN
 F 1 "10K" V 6850 4850 50  0000 C CNN
-F 2 "SM0402" H 6750 4700 60  0001 C CNN
+F 2 "0402" H 6750 4700 60  0001 C CNN
 F 4 "Panasonic - ECG" H 6750 4700 60  0001 C CNN "Manufacturer"
 F 5 "ERJ-2GEJ103X" H 6750 4700 60  0001 C CNN "Part Number"
@@
 $EndComp
 $Comp
-L R_US R?
+L R_US R28
 U 1 1 4F8F8AD9
 P 6750 2050
-F 0 "R?" V 6750 2150 50  0000 C CNN
+F 0 "R28" V 6750 2150 50  0000 C CNN
 F 1 "10K" V 6850 2200 50  0000 C CNN
-F 2 "SM0402" H 6750 2050 60  0001 C CNN
+F 2 "0402" H 6750 2050 60  0001 C CNN
 F 4 "Panasonic - ECG" H 6750 2050 60  0001 C CNN "Manufacturer"
 F 5 "ERJ-2GEJ103X" H 6750 2050 60  0001 C CNN "Part Number"
@@
 Wire Wire Line
 	6750 1600 6750 1800
+$Comp
+L OPA454AIDDA U8
+U 1 1 4F9A8E72
+P 5650 5350
+F 0 "U8" H 5650 5950 60  0000 C CNN
+F 1 "OPA454AIDDA" H 5650 4700 60  0000 C CNN
+F 2 "SOP_8_PowerPad_DDA" H 5650 5350 60  0001 C CNN
+F 4 "Texas Instruments" H 5650 5350 60  0001 C CNN "Manufacturer"
+F 5 "OPA454AIDDA" H 5650 5350 60  0001 C CNN "Part Number"
+F 6 "IC OPAMP GP 2.5MHZ SGL 8SOIC" H 5650 5350 60  0001 C CNN "Description"
+	1    5650 5350
+	1    0    0    -1
+$EndComp
 $EndSCHEMATC
