File: SCI-BREADBRD_vref.sch (KiCad schematic (older format))
At the start: 17 parts, among them P10 SF_ANLG, P11 SF_MOD, P12 CONN_1X2, U8 OPA454AIDDA, U9 OPA454AIDDA

Commit message: Completed ERC. Added some power flags and fixed mis-connected pins.
Changed lines of the file:
@@
-EESchema Schematic File Version 2  date Fri 27 Apr 2012 09:11:54 AM EDT
+EESchema Schematic File Version 2  date Fri 27 Apr 2012 11:11:24 AM EDT
 LIBS:custom_transistors
 LIBS:TI_custom
@@
 $EndDescr
 $Comp
-L AFE/SCI_ANLG_VDD #PWR075
+L AFE/SCI_ANLG_VDD #PWR083
 U 1 1 4F8F9D48
 P 4600 4350
-F 0 "#PWR075" H 4600 4450 30  0001 C CNN
+F 0 "#PWR083" H 4600 4450 30  0001 C CNN
 F 1 "AFE/SCI_ANLG_VDD" H 4600 4450 30  0000 C CNN
 	1    4600 4350
@@
 $EndComp
 $Comp
-L AFE/SCI_ANLG_VSS #PWR076
+L AFE/SCI_ANLG_VSS #PWR084
 U 1 1 4F8F9D57
 P 4650 6100
-F 0 "#PWR076" H 4650 6000 30  0001 C CNN
+F 0 "#PWR084" H 4650 6000 30  0001 C CNN
 F 1 "AFE/SCI_ANLG_VSS" H 4650 6000 30  0000 C CNN
 	1    4650 6100
@@
 $EndComp
 $Comp
-L GND #PWR077
+L GND #PWR085
 U 1 1 4F8FA231
 P 6400 5950
-F 0 "#PWR077" H 6400 5950 30  0001 C CNN
+F 0 "#PWR085" H 6400 5950 30  0001 C CNN
 F 1 "GND" H 6400 5880 30  0001 C CNN
 	1    6400 5950
@@
 $EndComp
 $Comp
-L GND #PWR078
+L GND #PWR086
 U 1 1 4F8FA8AC
 P 6450 3250
-F 0 "#PWR078" H 6450 3250 30  0001 C CNN
+F 0 "#PWR086" H 6450 3250 30  0001 C CNN
 F 1 "GND" H 6450 3180 30  0001 C CNN
 	1    6450 3250
@@
 $EndComp
 $Comp
-L MOD_VDD #PWR079
+L MOD_VDD #PWR087
 U 1 1 4F8FA8ED
 P 4650 1650
-F 0 "#PWR079" H 4650 1750 30  0001 C CNN
+F 0 "#PWR087" H 4650 1750 30  0001 C CNN
 F 1 "MOD_VDD" H 4650 1750 30  0000 C CNN
 	1    4650 1650
@@
 $EndComp
 $Comp
-L MOD_VSS #PWR080
+L MOD_VSS #PWR088
 U 1 1 4F8FA8FC
 P 4700 3400
-F 0 "#PWR080" H 4700 3300 30  0001 C CNN
+F 0 "#PWR088" H 4700 3300 30  0001 C CNN
 F 1 "MOD_VSS" H 4700 3300 30  0000 C CNN
 	1    4700 3400
@@
 $EndComp
 $Comp
-L SCI_DVDD_3_3V #PWR081
+L SCI_DVDD_3_3V #PWR089
 U 1 1 4F8FA967
 P 6450 1550
-F 0 "#PWR081" H 6450 1650 30  0001 C CNN
+F 0 "#PWR089" H 6450 1650 30  0001 C CNN
 F 1 "SCI_DVDD_3_3V" H 6450 1650 30  0000 C CNN
 	1    6450 1550
@@
 $EndComp
 $Comp
-L SCI_DVDD_3_3V #PWR082
+L SCI_DVDD_3_3V #PWR090
 U 1 1 4F8FA974
 P 6400 4250
-F 0 "#PWR082" H 6400 4350 30  0001 C CNN
+F 0 "#PWR090" H 6400 4350 30  0001 C CNN
 F 1 "SCI_DVDD_3_3V" H 6400 4350 30  0000 C CNN
 	1    6400 4250
@@
 $EndComp
 $Comp
-L GND #PWR083
+L GND #PWR091
 U 1 1 4F8F7B5C
 P 3950 2700
-F 0 "#PWR083" H 3950 2700 30  0001 C CNN
+F 0 "#PWR091" H 3950 2700 30  0001 C CNN
 F 1 "GND" H 3950 2630 30  0001 C CNN
 	1    3950 2700
@@
 $EndComp
 $Comp
-L GND #PWR084
+L GND #PWR092
 U 1 1 4F8F8028
 P 3750 5050
-F 0 "#PWR084" H 3750 5050 30  0001 C CNN
+F 0 "#PWR092" H 3750 5050 30  0001 C CNN
 F 1 "GND" H 3750 4980 30  0001 C CNN
 	1    3750 5050
@@
 $EndComp
 $Comp
-L GND #PWR085
+L GND #PWR093
 U 1 1 4F8F839D
 P 4100 3950
-F 0 "#PWR085" H 4100 3950 30  0001 C CNN
+F 0 "#PWR093" H 4100 3950 30  0001 C CNN
 F 1 "GND" H 4100 3880 30  0001 C CNN
 	1    4100 3950
@@
 $EndComp
 $Comp
-L GND #PWR086
+L GND #PWR094
 U 1 1 4F8F8442
 P 3900 6650
-F 0 "#PWR086" H 3900 6650 30  0001 C CNN
+F 0 "#PWR094" H 3900 6650 30  0001 C CNN
 F 1 "GND" H 3900 6580 30  0001 C CNN
 	1    3900 6650
@@
 	0    1    1    0
 $EndComp
-Wire Wire Line
-	4900 6050 3900 6050
-Wire Wire Line
-	4600 4350 4600 4900
-Wire Wire Line
-	4600 4900 5000 4900
-Wire Wire Line
-	4150 6050 4150 6000
-Wire Wire Line
-	4150 4900 4150 4450
-Connection ~ 4600 4450
-Wire Wire Line
-	4150 5400 4150 5500
-Wire Wire Line
-	4150 5450 5000 5450
-Connection ~ 4150 5450
-Connection ~ 4150 5450
-Connection ~ 4650 6050
-Wire Wire Line
-	4650 6050 4650 6050
-Wire Wire Line
-	5000 5700 4900 5700
-Wire Wire Line
-	4900 5700 4900 6050
-Wire Wire Line
-	5000 5850 4900 5850
-Connection ~ 4900 5850
-Wire Wire Line
-	4650 6100 4650 6050
-Wire Wire Line
-	5000 5250 4850 5250
-Wire Wire Line
-	4850 5250 4850 3950
-Wire Wire Line
-	4850 3950 7450 3950
-Wire Wire Line
-	7450 3300 7450 5350
-Wire Wire Line
-	6300 5850 6400 5850
-Wire Wire Line
-	6400 5850 6400 5950
-Wire Wire Line
-	7050 5050 7050 4950
-Wire Wire Line
-	6400 4250 6400 4350
-Wire Wire Line
-	6400 4850 6400 4900
-Wire Wire Line
-	6400 4900 6300 4900
-Wire Wire Line
-	4950 3350 4100 3350
-Wire Wire Line
-	4650 1650 4650 2200
-Wire Wire Line
-	4650 2200 5050 2200
-Wire Wire Line
-	4450 3350 4450 3300
-Wire Wire Line
-	4450 2200 4450 2100
-Wire Wire Line
-	4450 2700 4450 2800
-Wire Wire Line
-	4450 2750 5050 2750
-Connection ~ 4450 2750
-Connection ~ 4450 2750
-Connection ~ 4700 3350
-Wire Wire Line
-	4700 3350 4700 3350
-Wire Wire Line
-	5050 3000 4950 3000
-Wire Wire Line
-	4950 3000 4950 3350
-Wire Wire Line
-	5050 3150 4950 3150
-Connection ~ 4950 3150
-Wire Wire Line
-	4700 3400 4700 3350
-Wire Wire Line
-	5050 2550 4900 2550
-Wire Wire Line
-	4900 2550 4900 1250
-Wire Wire Line
-	4900 1250 7500 1250
-Wire Wire Line
-	7500 1250 7500 3100
-Wire Wire Line
-	6350 3150 6450 3150
-Wire Wire Line
-	6450 3150 6450 3250
-Wire Wire Line
-	7100 2350 7100 2250
-Wire Wire Line
-	6450 1550 6450 1650
-Wire Wire Line
-	6450 2150 6450 2200
-Wire Wire Line
-	6450 2200 6350 2200
-Wire Wire Line
-	7450 5350 6300 5350
-Wire Wire Line
-	7500 2650 6350 2650
-Wire Wire Line
-	7500 3100 7800 3100
-Connection ~ 7500 2650
-Wire Wire Line
-	7450 3300 7800 3300
-Connection ~ 7450 3950
-Wire Wire Line
-	3950 2700 3950 2600
-Wire Wire Line
-	3950 2200 3950 2100
-Wire Wire Line
-	3950 2100 4650 2100
-Connection ~ 4650 2100
-Connection ~ 4450 2100
-Wire Wire Line
-	3750 5050 3750 4950
-Wire Wire Line
-	3750 4550 3750 4450
-Wire Wire Line
-	3750 4450 4600 4450
-Connection ~ 4150 4450
-Connection ~ 4150 4450
-Wire Wire Line
-	4100 3950 4100 3850
-Wire Wire Line
-	4100 3350 4100 3450
-Connection ~ 4450 3350
-Wire Wire Line
-	3900 6650 3900 6550
-Wire Wire Line
-	3900 6050 3900 6150
-Connection ~ 4150 6050
-Wire Wire Line
-	6750 4450 6750 4300
-Wire Wire Line
-	6750 4300 6400 4300
-Connection ~ 6450 1600
-Wire Wire Line
-	6300 5050 7050 5050
-Wire Wire Line
-	6750 4950 6750 5050
-Connection ~ 6750 5050
-Wire Wire Line
-	6350 2350 7100 2350
-Wire Wire Line
-	6750 2350 6750 2300
-Connection ~ 6750 2350
-Wire Wire Line
-	6450 1600 6750 1600
-Wire Wire Line
-	6750 1600 6750 1800
 $Comp
 L OPA454AIDDA U8
@@
 	1    0    0    -1
 $EndComp
+Wire Wire Line
+	4900 6050 3900 6050
+Wire Wire Line
+	4600 4350 4600 4900
+Wire Wire Line
+	4600 4900 5000 4900
+Wire Wire Line
+	4150 6050 4150 6000
+Wire Wire Line
+	4150 4900 4150 4450
+Connection ~ 4600 4450
+Wire Wire Line
+	4150 5400 4150 5500
+Wire Wire Line
+	4150 5450 5000 5450
+Connection ~ 4150 5450
+Connection ~ 4150 5450
+Connection ~ 4650 6050
+Wire Wire Line
+	4650 6050 4650 6050
+Wire Wire Line
+	5000 5700 4900 5700
+Wire Wire Line
+	4900 5700 4900 6050
+Wire Wire Line
+	5000 5850 4900 5850
+Connection ~ 4900 5850
+Wire Wire Line
+	4650 6100 4650 6050
+Wire Wire Line
+	5000 5250 4850 5250
+Wire Wire Line
+	4850 5250 4850 3950
+Wire Wire Line
+	4850 3950 7450 3950
+Wire Wire Line
+	7450 3300 7450 5350
+Wire Wire Line
+	6300 5850 6400 5850
+Wire Wire Line
+	6400 5850 6400 5950
+Wire Wire Line
+	7050 5050 7050 4950
+Wire Wire Line
+	6400 4250 6400 4350
+Wire Wire Line
+	6400 4850 6400 4900
+Wire Wire Line
+	6400 4900 6300 4900
+Wire Wire Line
+	4950 3350 4100 3350
+Wire Wire Line
+	4650 1650 4650 2200
+Wire Wire Line
+	4650 2200 5050 2200
+Wire Wire Line
+	4450 3350 4450 3300
+Wire Wire Line
+	4450 2200 4450 2100
+Wire Wire Line
+	4450 2700 4450 2800
+Wire Wire Line
+	4450 2750 5050 2750
+Connection ~ 4450 2750
+Connection ~ 4450 2750
+Connection ~ 4700 3350
+Wire Wire Line
+	4700 3350 4700 3350
+Wire Wire Line
+	5050 3000 4950 3000
+Wire Wire Line
+	4950 3000 4950 3350
+Wire Wire Line
+	5050 3150 4950 3150
+Connection ~ 4950 3150
+Wire Wire Line
+	4700 3400 4700 3350
+Wire Wire Line
+	5050 2550 4900 2550
+Wire Wire Line
+	4900 2550 4900 1250
+Wire Wire Line
+	4900 1250 7500 1250
+Wire Wire Line
+	7500 1250 7500 3100
+Wire Wire Line
+	6350 3150 6450 3150
+Wire Wire Line
+	6450 3150 6450 3250
+Wire Wire Line
+	7100 2350 7100 2250
+Wire Wire Line
+	6450 1550 6450 1650
+Wire Wire Line
+	6450 2150 6450 2200
+Wire Wire Line
+	6450 2200 6350 2200
+Wire Wire Line
+	7450 5350 6300 5350
+Wire Wire Line
+	7500 2650 6350 2650
+Wire Wire Line
+	7500 3100 7800 3100
+Connection ~ 7500 2650
+Wire Wire Line
+	7450 3300 7800 3300
+Connection ~ 7450 3950
+Wire Wire Line
+	3950 2700 3950 2600
+Wire Wire Line
+	3950 2200 3950 2100
+Wire Wire Line
+	3950 2100 4650 2100
+Connection ~ 4650 2100
+Connection ~ 4450 2100
+Wire Wire Line
+	3750 5050 3750 4950
+Wire Wire Line
+	3750 4550 3750 4450
+Wire Wire Line
+	3750 4450 4600 4450
+Connection ~ 4150 4450
+Connection ~ 4150 4450
+Wire Wire Line
+	4100 3950 4100 3850
+Wire Wire Line
+	4100 3350 4100 3450
+Connection ~ 4450 3350
+Wire Wire Line
+	3900 6650 3900 6550
+Wire Wire Line
+	3900 6050 3900 6150
+Connection ~ 4150 6050
+Wire Wire Line
+	6750 4450 6750 4300
+Connection ~ 6450 1600
+Wire Wire Line
+	6300 5050 7050 5050
+Wire Wire Line
+	6750 4950 6750 5050
+Connection ~ 6750 5050
+Wire Wire Line
+	6350 2350 7100 2350
+Wire Wire Line
+	6750 2350 6750 2300
+Connection ~ 6750 2350
+Wire Wire Line
+	6450 1600 6750 1600
+Wire Wire Line
+	6750 1600 6750 1800
+Wire Wire Line
+	6750 4300 6400 4300
+Connection ~ 6400 4300
 $EndSCHEMATC

Commit message: Changed the testpoints to have a refdes of TP? instead of P? and re-annotated.
Fixed a but in better_bom that was causing the last field to be
erroneous.

Added the -e option to better_bom to allow excluding fields
Parts:
- removed P10: SF_ANLG, TESTVIA_p30mil_h20mil, symbol TST
- removed P11: SF_MOD, TESTVIA_p30mil_h20mil, symbol TST
- added P10, P11: TP, TESTVIA_p30mil_h20mil, symbol TP
Connections:
- wire segments 66 -> 84
Changed lines of the file:
@@
-EESchema Schematic File Version 2  date Fri 27 Apr 2012 11:11:24 AM EDT
+EESchema Schematic File Version 2  date Fri 27 Apr 2012 01:15:52 PM EDT
 LIBS:custom_transistors
 LIBS:TI_custom
@@
 $EndDescr
 $Comp
-L AFE/SCI_ANLG_VDD #PWR083
+L AFE/SCI_ANLG_VDD #PWR81
 U 1 1 4F8F9D48
 P 4600 4350
-F 0 "#PWR083" H 4600 4450 30  0001 C CNN
+F 0 "#PWR81" H 4600 4450 30  0001 C CNN
 F 1 "AFE/SCI_ANLG_VDD" H 4600 4450 30  0000 C CNN
 	1    4600 4350
@@
 $EndComp
 $Comp
-L AFE/SCI_ANLG_VSS #PWR084
+L AFE/SCI_ANLG_VSS #PWR83
 U 1 1 4F8F9D57
 P 4650 6100
-F 0 "#PWR084" H 4650 6000 30  0001 C CNN
+F 0 "#PWR83" H 4650 6000 30  0001 C CNN
 F 1 "AFE/SCI_ANLG_VSS" H 4650 6000 30  0000 C CNN
 	1    4650 6100
@@
 $EndComp
 $Comp
-L GND #PWR085
+L GND #PWR86
 U 1 1 4F8FA231
 P 6400 5950
-F 0 "#PWR085" H 6400 5950 30  0001 C CNN
+F 0 "#PWR86" H 6400 5950 30  0001 C CNN
 F 1 "GND" H 6400 5880 30  0001 C CNN
 	1    6400 5950
-	1    0    0    -1
-$EndComp
-$Comp
-L TST P10
-U 1 1 4F8FA275
-P 7050 4950
-F 0 "P10" H 7050 5250 40  0000 C CNN
-F 1 "SF_ANLG" H 7050 5200 30  0000 C CNN
-F 2 "TESTVIA_p30mil_h20mil" H 7050 4950 60  0001 C CNN
-F 4 "TESTPOINT VIA" H 7050 4950 60  0001 C CNN "Description"
-F 5 "NO PART. TEST PAD ONLY" H 7050 4950 60  0001 C CNN "Note"
-	1    7050 4950
 	1    0    0    -1
 $EndComp
@@
 $EndComp
 $Comp
-L GND #PWR086
+L GND #PWR88
 U 1 1 4F8FA8AC
 P 6450 3250
-F 0 "#PWR086" H 6450 3250 30  0001 C CNN
+F 0 "#PWR88" H 6450 3250 30  0001 C CNN
 F 1 "GND" H 6450 3180 30  0001 C CNN
 	1    6450 3250
-	1    0    0    -1
-$EndComp
-$Comp
-L TST P11
-U 1 1 4F8FA8B4
-P 7100 2250
-F 0 "P11" H 7100 2550 40  0000 C CNN
-F 1 "SF_MOD" H 7100 2500 30  0000 C CNN
-F 2 "TESTVIA_p30mil_h20mil" H 7100 2250 60  0001 C CNN
-F 4 "TESTPOINT VIA" H 7100 2250 60  0001 C CNN "Description"
-F 5 "NO PART. TEST PAD ONLY" H 7100 2250 60  0001 C CNN "Note"
-	1    7100 2250
 	1    0    0    -1
 $EndComp
@@
 $EndComp
 $Comp
-L MOD_VDD #PWR087
+L MOD_VDD #PWR82
 U 1 1 4F8FA8ED
 P 4650 1650
-F 0 "#PWR087" H 4650 1750 30  0001 C CNN
+F 0 "#PWR82" H 4650 1750 30  0001 C CNN
 F 1 "MOD_VDD" H 4650 1750 30  0000 C CNN
 	1    4650 1650
@@
 $EndComp
 $Comp
-L MOD_VSS #PWR088
+L MOD_VSS #PWR84
 U 1 1 4F8FA8FC
 P 4700 3400
-F 0 "#PWR088" H 4700 3300 30  0001 C CNN
+F 0 "#PWR84" H 4700 3300 30  0001 C CNN
 F 1 "MOD_VSS" H 4700 3300 30  0000 C CNN
 	1    4700 3400
@@
 $EndComp
 $Comp
-L SCI_DVDD_3_3V #PWR089
+L SCI_DVDD_3_3V #PWR87
 U 1 1 4F8FA967
 P 6450 1550
-F 0 "#PWR089" H 6450 1650 30  0001 C CNN
+F 0 "#PWR87" H 6450 1650 30  0001 C CNN
 F 1 "SCI_DVDD_3_3V" H 6450 1650 30  0000 C CNN
 	1    6450 1550
@@
 $EndComp
 $Comp
-L SCI_DVDD_3_3V #PWR090
+L SCI_DVDD_3_3V #PWR85
 U 1 1 4F8FA974
 P 6400 4250
-F 0 "#PWR090" H 6400 4350 30  0001 C CNN
+F 0 "#PWR85" H 6400 4350 30  0001 C CNN
 F 1 "SCI_DVDD_3_3V" H 6400 4350 30  0000 C CNN
 	1    6400 4250
@@
 $EndComp
 $Comp
-L GND #PWR091
+L GND #PWR79
 U 1 1 4F8F7B5C
 P 3950 2700
-F 0 "#PWR091" H 3950 2700 30  0001 C CNN
+F 0 "#PWR79" H 3950 2700 30  0001 C CNN
 F 1 "GND" H 3950 2630 30  0001 C CNN
 	1    3950 2700
@@
 $EndComp
 $Comp
-L GND #PWR092
+L GND #PWR77
 U 1 1 4F8F8028
 P 3750 5050
-F 0 "#PWR092" H 3750 5050 30  0001 C CNN
+F 0 "#PWR77" H 3750 5050 30  0001 C CNN
 F 1 "GND" H 3750 4980 30  0001 C CNN
 	1    3750 5050
@@
 $EndComp
 $Comp
-L GND #PWR093
+L GND #PWR80
 U 1 1 4F8F839D
 P 4100 3950
-F 0 "#PWR093" H 4100 3950 30  0001 C CNN
+F 0 "#PWR80" H 4100 3950 30  0001 C CNN
 F 1 "GND" H 4100 3880 30  0001 C CNN
 	1    4100 3950
@@
 $EndComp
 $Comp
-L GND #PWR094
+L GND #PWR78
 U 1 1 4F8F8442
 P 3900 6650
-F 0 "#PWR094" H 3900 6650 30  0001 C CNN
+F 0 "#PWR78" H 3900 6650 30  0001 C CNN
 F 1 "GND" H 3900 6580 30  0001 C CNN
 	1    3900 6650
@@
 $EndComp
 Wire Wire Line
-	4900 6050 3900 6050
-Wire Wire Line
-	4600 4350 4600 4900
+	4900 6050 4650 6050
+Wire Wire Line
+	4650 6050 4150 6050
+Wire Wire Line
+	4150 6050 3900 6050
+Wire Wire Line
+	4600 4350 4600 4450
+Wire Wire Line
+	4600 4450 4600 4900
 Wire Wire Line
 	4600 4900 5000 4900
@@
 Connection ~ 4600 4450
 Wire Wire Line
-	4150 5400 4150 5500
+	4150 5400 4150 5450
+Wire Wire Line
+	4150 5450 4150 5500
 Wire Wire Line
 	4150 5450 5000 5450
@@
 	5000 5700 4900 5700
 Wire Wire Line
-	4900 5700 4900 6050
+	4900 5700 4900 5850
+Wire Wire Line
+	4900 5850 4900 6050
 Wire Wire Line
 	5000 5850 4900 5850
@@
 	4850 3950 7450 3950
 Wire Wire Line
-	7450 3300 7450 5350
+	7450 3300 7450 3950
+Wire Wire Line
+	7450 3950 7450 5350
 Wire Wire Line
 	6300 5850 6400 5850
@@
 	6400 5850 6400 5950
 Wire Wire Line
-	7050 5050 7050 4950
-Wire Wire Line
-	6400 4250 6400 4350
+	7200 5050 7200 4950
+Wire Wire Line
+	6400 4250 6400 4300
+Wire Wire Line
+	6400 4300 6400 4350
 Wire Wire Line
 	6400 4850 6400 4900
@@
 	6400 4900 6300 4900
 Wire Wire Line
-	4950 3350 4100 3350
-Wire Wire Line
-	4650 1650 4650 2200
+	4950 3350 4700 3350
+Wire Wire Line
+	4700 3350 4450 3350
+Wire Wire Line
+	4450 3350 4100 3350
+Wire Wire Line
+	4650 1650 4650 2100
+Wire Wire Line
+	4650 2100 4650 2200
 Wire Wire Line
 	4650 2200 5050 2200
@@
 	4450 2200 4450 2100
 Wire Wire Line
-	4450 2700 4450 2800
+	4450 2700 4450 2750
+Wire Wire Line
+	4450 2750 4450 2800
 Wire Wire Line
 	4450 2750 5050 2750
@@
 	5050 3000 4950 3000
 Wire Wire Line
-	4950 3000 4950 3350
+	4950 3000 4950 3150
+Wire Wire Line
+	4950 3150 4950 3350
 Wire Wire Line
 	5050 3150 4950 3150
@@
 	4900 1250 7500 1250
 Wire Wire Line
-	7500 1250 7500 3100
+	7500 1250 7500 2650
+Wire Wire Line
+	7500 2650 7500 3100
 Wire Wire Line
 	6350 3150 6450 3150
@@
 	6450 3150 6450 3250
 Wire Wire Line
-	7100 2350 7100 2250
-Wire Wire Line
-	6450 1550 6450 1650
+	7200 2350 7200 2250
+Wire Wire Line
+	6450 1550 6450 1600
+Wire Wire Line
+	6450 1600 6450 1650
 Wire Wire Line
 	6450 2150 6450 2200
@@
 	3950 2200 3950 2100
 Wire Wire Line
-	3950 2100 4650 2100
+	3950 2100 4450 2100
+Wire Wire Line
+	4450 2100 4650 2100
 Connection ~ 4650 2100
 Connection ~ 4450 2100
@@
 	3750 4550 3750 4450
 Wire Wire Line
-	3750 4450 4600 4450
+	3750 4450 4150 4450
+Wire Wire Line
+	4150 4450 4600 4450
 Connection ~ 4150 4450
 Connection ~ 4150 4450
@@
 Connection ~ 6450 1600
 Wire Wire Line
-	6300 5050 7050 5050
+	6300 5050 6750 5050
+Wire Wire Line
+	6750 5050 7200 5050
 Wire Wire Line
 	6750 4950 6750 5050
 Connection ~ 6750 5050
 Wire Wire Line
-	6350 2350 7100 2350
+	6350 2350 6750 2350
+Wire Wire Line
+	6750 2350 7200 2350
 Wire Wire Line
 	6750 2350 6750 2300
@@
 	6750 4300 6400 4300
 Connection ~ 6400 4300
+$Comp
+L TP P10
+U 1 1 4F9AD9B8
+P 7200 2250
+F 0 "P10" H 7200 2600 40  0000 C CNN
+F 1 "TP" H 7200 2500 30  0001 C CNN
+F 2 "TESTVIA_p30mil_h20mil" H 7200 2250 60  0001 C CNN
+F 4 "TESTPOINT VIA" H 7200 2250 60  0001 C CNN "Description"
+F 5 "NO PART. TEST PAD ONLY." H 7200 2250 60  0001 C CNN "Note"
+F 6 "SF_MOD" H 7200 2500 60  0000 C CNN "Silkscreen"
+	1    7200 2250
+	1    0    0    -1
+$EndComp
+$Comp
+L TP P11
+U 1 1 4F9AD9F2
+P 7200 4950
+F 0 "P11" H 7200 5300 40  0000 C CNN
+F 1 "TP" H 7200 5200 30  0001 C CNN
+F 2 "TESTVIA_p30mil_h20mil" H 7200 4950 60  0001 C CNN
+F 4 "TESTPOINT VIA" H 7200 4950 60  0001 C CNN "Description"
+F 5 "NO PART. TEST PAD ONLY." H 7200 4950 60  0001 C CNN "Note"
+F 6 "SF_ANLG" H 7200 5200 60  0000 C CNN "Silkscreen"
+	1    7200 4950
+	1    0    0    -1
+$EndComp
 $EndSCHEMATC

Commit message: Enlarged the text on all of the power rails to make them easier to see when plotted
Other:
- moved on the sheet: C17, C18, C19, C20, R22, R23, R24, R25

Commit message: Re-annotated for added parts.
Connections:
- wire segments 84 -> 64
Changed lines of the file:
@@
-EESchema Schematic File Version 2  date Fri 27 Apr 2012 02:46:40 PM EDT
+EESchema Schematic File Version 2  date Wed 02 May 2012 02:37:03 AM EDT
 LIBS:custom_transistors
 LIBS:TI_custom
@@
 Sheet 9 9
 Title "SCI-BREADBRD-MVK"
-Date "27 apr 2012"
+Date "2 may 2012"
 Rev "A"
 Comp "The Ohio State University"
@@
 $EndComp
 $Comp
-L GND #PWR86
+L GND #PWR083
 U 1 1 4F8FA231
 P 6400 5950
-F 0 "#PWR86" H 6400 5950 30  0001 C CNN
+F 0 "#PWR083" H 6400 5950 30  0001 C CNN
 F 1 "GND" H 6400 5880 30  0001 C CNN
 	1    6400 5950
@@
 $EndComp
 $Comp
-L GND #PWR88
+L GND #PWR084
 U 1 1 4F8FA8AC
 P 6450 3250
-F 0 "#PWR88" H 6450 3250 30  0001 C CNN
+F 0 "#PWR084" H 6450 3250 30  0001 C CNN
 F 1 "GND" H 6450 3180 30  0001 C CNN
 	1    6450 3250
@@
 $EndComp
 $Comp
-L GND #PWR79
+L GND #PWR085
 U 1 1 4F8F7B5C
 P 3800 2700
-F 0 "#PWR79" H 3800 2700 30  0001 C CNN
+F 0 "#PWR085" H 3800 2700 30  0001 C CNN
 F 1 "GND" H 3800 2630 30  0001 C CNN
 	1    3800 2700
@@
 $EndComp
 $Comp
-L GND #PWR77
+L GND #PWR086
 U 1 1 4F8F8028
 P 3500 5050
-F 0 "#PWR77" H 3500 5050 30  0001 C CNN
+F 0 "#PWR086" H 3500 5050 30  0001 C CNN
 F 1 "GND" H 3500 4980 30  0001 C CNN
 	1    3500 5050
@@
 $EndComp
 $Comp
-L GND #PWR80
+L GND #PWR087
 U 1 1 4F8F839D
 P 3950 3950
-F 0 "#PWR80" H 3950 3950 30  0001 C CNN
+F 0 "#PWR087" H 3950 3950 30  0001 C CNN
 F 1 "GND" H 3950 3880 30  0001 C CNN
 	1    3950 3950
@@
 $EndComp
 $Comp
-L GND #PWR78
+L GND #PWR088
 U 1 1 4F8F8442
 P 3650 6650
-F 0 "#PWR78" H 3650 6650 30  0001 C CNN
+F 0 "#PWR088" H 3650 6650 30  0001 C CNN
 F 1 "GND" H 3650 6580 30  0001 C CNN
 	1    3650 6650
@@
 $EndComp
 Wire Wire Line
-	4900 6050 4400 6050
-Wire Wire Line
-	4400 6050 3900 6050
-Wire Wire Line
-	3900 6050 3650 6050
-Wire Wire Line
-	4350 4350 4350 4450
-Wire Wire Line
-	4350 4450 4350 4900
+	4900 6050 3650 6050
+Wire Wire Line
+	4350 4350 4350 4900
 Wire Wire Line
 	4350 4900 5000 4900
@@
 Connection ~ 4350 4450
 Wire Wire Line
-	3900 5400 3900 5450
-Wire Wire Line
-	3900 5450 3900 5500
+	3900 5400 3900 5500
 Wire Wire Line
 	3900 5450 5000 5450
@@
 	5000 5700 4900 5700
 Wire Wire Line
-	4900 5700 4900 5850
-Wire Wire Line
-	4900 5850 4900 6050
+	4900 5700 4900 6200
 Wire Wire Line
 	5000 5850 4900 5850
 Connection ~ 4900 5850
 Wire Wire Line
-	4900 6200 4900 6050
-Wire Wire Line
 	5000 5250 4850 5250
 Wire Wire Line
@@
 	4850 3950 7450 3950
 Wire Wire Line
-	7450 3300 7450 3950
-Wire Wire Line
-	7450 3950 7450 5350
+	7450 3300 7450 5350
 Wire Wire Line
 	6300 5850 6400 5850
@@
 	7200 5050 7200 4950
 Wire Wire Line
-	6400 4250 6400 4300
-Wire Wire Line
-	6400 4300 6400 4350
+	6400 4250 6400 4350
 Wire Wire Line
 	6400 4850 6400 4900
@@
 	6400 4900 6300 4900
 Wire Wire Line
-	4950 3350 4550 3350
-Wire Wire Line
-	4550 3350 4300 3350
-Wire Wire Line
-	4300 3350 3950 3350
-Wire Wire Line
-	4500 1650 4500 2100
-Wire Wire Line
-	4500 2100 4500 2200
+	4950 3350 3950 3350
+Wire Wire Line
+	4500 1650 4500 2200
 Wire Wire Line
 	4500 2200 5050 2200
@@
 	4300 2200 4300 2100
 Wire Wire Line
-	4300 2700 4300 2750
-Wire Wire Line
-	4300 2750 4300 2800
+	4300 2700 4300 2800
 Wire Wire Line
 	4300 2750 5050 2750
@@
 	5050 3000 4950 3000
 Wire Wire Line
-	4950 3000 4950 3150
-Wire Wire Line
-	4950 3150 4950 3350
+	4950 3000 4950 3550
 Wire Wire Line
 	5050 3150 4950 3150
 Connection ~ 4950 3150
 Wire Wire Line
-	4950 3550 4950 3350
-Wire Wire Line
 	5050 2550 4900 2550
 Wire Wire Line
@@
 	4900 1250 7500 1250
 Wire Wire Line
-	7500 1250 7500 2650
-Wire Wire Line
-	7500 2650 7500 3100
+	7500 1250 7500 3100
 Wire Wire Line
 	6350 3150 6450 3150
@@
 	7200 2350 7200 2250
 Wire Wire Line
-	6450 1550 6450 1600
-Wire Wire Line
-	6450 1600 6450 1650
+	6450 1550 6450 1650
 Wire Wire Line
 	6450 2150 6450 2200
@@
 	3800 2200 3800 2100
 Wire Wire Line
-	3800 2100 4300 2100
-Wire Wire Line
-	4300 2100 4500 2100
+	3800 2100 4500 2100
 Connection ~ 4500 2100
 Connection ~ 4300 2100
@@
 	3500 4550 3500 4450
 Wire Wire Line
-	3500 4450 3900 4450
-Wire Wire Line
-	3900 4450 4350 4450
+	3500 4450 4350 4450
 Connection ~ 3900 4450
 Connection ~ 3900 4450
@@
 Connection ~ 6450 1600
 Wire Wire Line
-	6300 5050 6750 5050
-Wire Wire Line
-	6750 5050 7200 5050
+	6300 5050 7200 5050
 Wire Wire Line
 	6750 4950 6750 5050
 Connection ~ 6750 5050
 Wire Wire Line
-	6350 2350 6750 2350
-Wire Wire Line
-	6750 2350 7200 2350
+	6350 2350 7200 2350
 Wire Wire Line
 	6750 2350 6750 2300
@@
 $EndComp
 $Comp
-L MOD_VDD #PWR?
+L MOD_VDD #PWR089
 U 1 1 4F9AECA0
 P 4500 1650
-F 0 "#PWR?" H 4500 1750 30  0001 C CNN
+F 0 "#PWR089" H 4500 1750 30  0001 C CNN
 F 1 "MOD_VDD" H 4500 1800 60  0000 C CNN
 	1    4500 1650
@@
 $EndComp
 $Comp
-L MOD_VSS #PWR?
+L MOD_VSS #PWR090
 U 1 1 4F9AECAF
 P 4950 3550
-F 0 "#PWR?" H 4950 3450 30  0001 C CNN
+F 0 "#PWR090" H 4950 3450 30  0001 C CNN
 F 1 "MOD_VSS" H 4950 3400 60  0000 C CNN
 	1    4950 3550
@@
 $EndComp
 $Comp
-L SCI_DVDD_3_3V #PWR?
+L SCI_DVDD_3_3V #PWR091
 U 1 1 4F9AECC8
 P 6450 1550
-F 0 "#PWR?" H 6450 1650 30  0001 C CNN
+F 0 "#PWR091" H 6450 1650 30  0001 C CNN
 F 1 "SCI_DVDD_3_3V" H 6450 1700 60  0000 C CNN
 	1    6450 1550
@@
 $EndComp
 $Comp
-L SCI_DVDD_3_3V #PWR?
+L SCI_DVDD_3_3V #PWR092
 U 1 1 4F9AECD7
 P 6400 4250
-F 0 "#PWR?" H 6400 4350 30  0001 C CNN
+F 0 "#PWR092" H 6400 4350 30  0001 C CNN
 F 1 "SCI_DVDD_3_3V" H 6400 4400 60  0000 C CNN
 	1    6400 4250
@@
 $EndComp
 $Comp
-L AFE/SCI_ANLG_VDD #PWR?
+L AFE/SCI_ANLG_VDD #PWR093
 U 1 1 4F9AECE6
 P 4350 4350
-F 0 "#PWR?" H 4350 4450 30  0001 C CNN
+F 0 "#PWR093" H 4350 4450 30  0001 C CNN
 F 1 "AFE/SCI_ANLG_VDD" H 4350 4450 60  0000 C CNN
 	1    4350 4350
@@
 $EndComp
 $Comp
-L AFE/SCI_ANLG_VSS #PWR?
+L AFE/SCI_ANLG_VSS #PWR094
 U 1 1 4F9AECF5
 P 4900 6200
-F 0 "#PWR?" H 4900 6100 30  0001 C CNN
+F 0 "#PWR094" H 4900 6100 30  0001 C CNN
 F 1 "AFE/SCI_ANLG_VSS" H 4900 6050 60  0000 C CNN
 	1    4900 6200
