File: SCI-BREADBRD_avss.sch (KiCad schematic (older format))
At the start: 21 parts, among them P9 AVSS, U6 TPS63700DRC, U7 TPS72325DBV

Commit message: Completed ERC. Added some power flags and fixed mis-connected pins.
Connections:
- wire segments 58 -> 60
Other:
- moved on the sheet: C14, C8, C9, R16, R17

Commit message: Changed the testpoints to have a refdes of TP? instead of P? and re-annotated.
Fixed a but in better_bom that was causing the last field to be
erroneous.

Added the -e option to better_bom to allow excluding fields
Parts:
- removed P9: AVSS, TESTVIA_p30mil_h20mil, symbol TST
- added P9: TP, TESTVIA_p30mil_h20mil, symbol TP
Changed lines of the file:
@@
-EESchema Schematic File Version 2  date Fri 27 Apr 2012 11:11:24 AM EDT
+EESchema Schematic File Version 2  date Fri 27 Apr 2012 01:15:52 PM EDT
 LIBS:custom_transistors
 LIBS:TI_custom
@@
 $Descr A4 11693 8268
 encoding utf-8
-Sheet 5 9
+Sheet 8 9
 Title "SCI-BREADBRD-MVK"
 Date "27 apr 2012"
@@
 $EndComp
 $Comp
-L GND #PWR069
+L GND #PWR68
 U 1 1 4F9A3367
 P 2750 4400
-F 0 "#PWR069" H 2750 4400 30  0001 C CNN
+F 0 "#PWR68" H 2750 4400 30  0001 C CNN
 F 1 "GND" H 2750 4330 30  0001 C CNN
 	1    2750 4400
@@
 $EndComp
 $Comp
-L SCI_AVDD_5_5V #PWR070
+L SCI_AVDD_5_5V #PWR65
 U 1 1 4F9A3376
 P 750 2650
-F 0 "#PWR070" H 750 2750 30  0001 C CNN
+F 0 "#PWR65" H 750 2750 30  0001 C CNN
 F 1 "SCI_AVDD_5_5V" H 750 2750 30  0000 C CNN
 	1    750  2650
@@
 $EndComp
 $Comp
-L GND #PWR071
+L GND #PWR66
 U 1 1 4F9A3385
 P 750 3750
-F 0 "#PWR071" H 750 3750 30  0001 C CNN
+F 0 "#PWR66" H 750 3750 30  0001 C CNN
 F 1 "GND" H 750 3680 30  0001 C CNN
 	1    750  3750
@@
 $EndComp
 $Comp
-L GND #PWR072
+L GND #PWR67
 U 1 1 4F9A339D
 P 1200 4400
-F 0 "#PWR072" H 1200 4400 30  0001 C CNN
+F 0 "#PWR67" H 1200 4400 30  0001 C CNN
 F 1 "GND" H 1200 4330 30  0001 C CNN
 	1    1200 4400
@@
 $EndComp
 $Comp
-L GND #PWR073
+L GND #PWR70
 U 1 1 4F9A33EB
 P 5200 3300
-F 0 "#PWR073" H 5200 3300 30  0001 C CNN
+F 0 "#PWR70" H 5200 3300 30  0001 C CNN
 F 1 "GND" H 5200 3230 30  0001 C CNN
 	1    5200 3300
@@
 $EndComp
 $Comp
-L GND #PWR074
+L GND #PWR69
 U 1 1 4F9A33F1
 P 4700 5050
-F 0 "#PWR074" H 4700 5050 30  0001 C CNN
+F 0 "#PWR69" H 4700 5050 30  0001 C CNN
 F 1 "GND" H 4700 4980 30  0001 C CNN
 	1    4700 5050
@@
 $EndComp
 $Comp
-L GND #PWR075
+L GND #PWR71
 U 1 1 4F9A3400
 P 5400 5050
-F 0 "#PWR075" H 5400 5050 30  0001 C CNN
+F 0 "#PWR71" H 5400 5050 30  0001 C CNN
 F 1 "GND" H 5400 4980 30  0001 C CNN
 	1    5400 5050
@@
 $EndComp
 $Comp
-L GND #PWR076
+L GND #PWR72
 U 1 1 4F9A340F
 P 7000 3950
-F 0 "#PWR076" H 7000 3950 30  0001 C CNN
+F 0 "#PWR72" H 7000 3950 30  0001 C CNN
 F 1 "GND" H 7000 3880 30  0001 C CNN
 	1    7000 3950
@@
 $EndComp
 $Comp
-L GND #PWR077
+L GND #PWR75
 U 1 1 4F9A341E
 P 9200 3750
-F 0 "#PWR077" H 9200 3750 30  0001 C CNN
+F 0 "#PWR75" H 9200 3750 30  0001 C CNN
 F 1 "GND" H 9200 3680 30  0001 C CNN
 	1    9200 3750
@@
 $EndComp
 $Comp
-L GND #PWR078
+L GND #PWR73
 U 1 1 4F9A3424
 P 7600 3900
-F 0 "#PWR078" H 7600 3900 30  0001 C CNN
+F 0 "#PWR73" H 7600 3900 30  0001 C CNN
 F 1 "GND" H 7600 3830 30  0001 C CNN
 	1    7600 3900
@@
 $EndComp
 $Comp
-L GND #PWR079
+L GND #PWR74
 U 1 1 4F9A3433
 P 8950 4350
-F 0 "#PWR079" H 8950 4350 30  0001 C CNN
+F 0 "#PWR74" H 8950 4350 30  0001 C CNN
 F 1 "GND" H 8950 4280 30  0001 C CNN
 	1    8950 4350
@@
 $EndComp
 $Comp
-L GND #PWR080
+L GND #PWR76
 U 1 1 4F9A344B
 P 9800 4350
-F 0 "#PWR080" H 9800 4350 30  0001 C CNN
+F 0 "#PWR76" H 9800 4350 30  0001 C CNN
 F 1 "GND" H 9800 4280 30  0001 C CNN
 	1    9800 4350
-	1    0    0    -1
-$EndComp
-$Comp
-L TST P9
-U 1 1 4F9A3453
-P 10100 3100
-F 0 "P9" H 10100 3400 40  0000 C CNN
-F 1 "AVSS" H 10100 3350 30  0000 C CNN
-F 2 "TESTVIA_p30mil_h20mil" H 10100 3100 60  0001 C CNN
-F 4 "TESTPOINT VIA" H 10100 3100 60  0001 C CNN "Description"
-F 5 "NO PART. TEST PAD ONLY." H 10100 3100 60  0001 C CNN "Note"
-	1    10100 3100
 	1    0    0    -1
 $EndComp
@@
 VSS_EN
 $Comp
-L PWR_FLAG #FLG081
+L PWR_FLAG #FLG6
 U 1 1 4F9AE33C
 P 1850 3150
-F 0 "#FLG081" H 1850 3245 30  0001 C CNN
+F 0 "#FLG6" H 1850 3245 30  0001 C CNN
 F 1 "PWR_FLAG" H 1850 3330 30  0000 C CNN
 	1    1850 3150
@@
 $EndComp
 $Comp
-L PWR_FLAG #FLG082
+L PWR_FLAG #FLG5
 U 1 1 4F9AE3FD
 P 1650 3750
-F 0 "#FLG082" H 1650 3845 30  0001 C CNN
+F 0 "#FLG5" H 1650 3845 30  0001 C CNN
 F 1 "PWR_FLAG" H 1650 3930 30  0000 C CNN
 	1    1650 3750
@@
 	1650 3750 1650 3900
 Connection ~ 1650 3900
+$Comp
+L TP P9
+U 1 1 4F9AD953
+P 10100 3100
+F 0 "P9" H 10100 3450 40  0000 C CNN
+F 1 "TP" H 10100 3350 30  0001 C CNN
+F 2 "TESTVIA_p30mil_h20mil" H 10100 3100 60  0001 C CNN
+F 4 "TESTPOINT VIA" H 10100 3100 60  0001 C CNN "Description"
+F 5 "NO PART. TEST PAD ONLY." H 10100 3100 60  0001 C CNN "Note"
+F 6 "AVSS" H 10100 3350 60  0000 C CNN "Silkscreen"
+	1    10100 3100
+	1    0    0    -1
+$EndComp
 $EndSCHEMATC

Commit message: Enlarged the text on all of the power rails to make them easier to see when plotted
Other:
- moved on the sheet: C10, C11, C12, C13, C14, C15, C16, C8, C9, D5, D6, L2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

Commit message: Added some bypass caps. Rearranged pins on connectors to make layout easier.
Parts:
- removed P9: TP, TESTVIA_p30mil_h20mil, symbol TP
Changed lines of the file:
@@
-EESchema Schematic File Version 2  date Wed 02 May 2012 02:37:03 AM EDT
+EESchema Schematic File Version 2  date Wed 02 May 2012 11:11:08 PM EDT
 LIBS:custom_transistors
 LIBS:TI_custom
@@
 Sheet 8 9
 Title "SCI-BREADBRD-MVK"
-Date "2 may 2012"
+Date "3 may 2012"
 Rev "A"
 Comp "The Ohio State University"
@@
 $EndComp
 $Comp
-L GND #PWR069
+L GND #PWR068
 U 1 1 4F9A3367
 P 2900 4400
-F 0 "#PWR069" H 2900 4400 30  0001 C CNN
+F 0 "#PWR068" H 2900 4400 30  0001 C CNN
 F 1 "GND" H 2900 4330 30  0001 C CNN
 	1    2900 4400
@@
 $EndComp
 $Comp
-L GND #PWR070
+L GND #PWR069
 U 1 1 4F9A3385
 P 900 3750
-F 0 "#PWR070" H 900 3750 30  0001 C CNN
+F 0 "#PWR069" H 900 3750 30  0001 C CNN
 F 1 "GND" H 900 3680 30  0001 C CNN
 	1    900  3750
@@
 $EndComp
 $Comp
-L GND #PWR071
+L GND #PWR070
 U 1 1 4F9A339D
 P 1350 4400
-F 0 "#PWR071" H 1350 4400 30  0001 C CNN
+F 0 "#PWR070" H 1350 4400 30  0001 C CNN
 F 1 "GND" H 1350 4330 30  0001 C CNN
 	1    1350 4400
@@
 $EndComp
 $Comp
-L GND #PWR072
+L GND #PWR071
 U 1 1 4F9A33EB
 P 5350 3300
-F 0 "#PWR072" H 5350 3300 30  0001 C CNN
+F 0 "#PWR071" H 5350 3300 30  0001 C CNN
 F 1 "GND" H 5350 3230 30  0001 C CNN
 	1    5350 3300
@@
 $EndComp
 $Comp
-L GND #PWR073
+L GND #PWR072
 U 1 1 4F9A33F1
 P 4850 5050
-F 0 "#PWR073" H 4850 5050 30  0001 C CNN
+F 0 "#PWR072" H 4850 5050 30  0001 C CNN
 F 1 "GND" H 4850 4980 30  0001 C CNN
 	1    4850 5050
@@
 $EndComp
 $Comp
-L GND #PWR074
+L GND #PWR073
 U 1 1 4F9A3400
 P 5550 5050
-F 0 "#PWR074" H 5550 5050 30  0001 C CNN
+F 0 "#PWR073" H 5550 5050 30  0001 C CNN
 F 1 "GND" H 5550 4980 30  0001 C CNN
 	1    5550 5050
@@
 $EndComp
 $Comp
-L GND #PWR075
+L GND #PWR074
 U 1 1 4F9A340F
 P 7150 3950
-F 0 "#PWR075" H 7150 3950 30  0001 C CNN
+F 0 "#PWR074" H 7150 3950 30  0001 C CNN
 F 1 "GND" H 7150 3880 30  0001 C CNN
 	1    7150 3950
@@
 $EndComp
 $Comp
-L GND #PWR076
+L GND #PWR075
 U 1 1 4F9A341E
 P 9350 3750
-F 0 "#PWR076" H 9350 3750 30  0001 C CNN
+F 0 "#PWR075" H 9350 3750 30  0001 C CNN
 F 1 "GND" H 9350 3680 30  0001 C CNN
 	1    9350 3750
@@
 $EndComp
 $Comp
-L GND #PWR077
+L GND #PWR076
 U 1 1 4F9A3424
 P 7750 3900
-F 0 "#PWR077" H 7750 3900 30  0001 C CNN
+F 0 "#PWR076" H 7750 3900 30  0001 C CNN
 F 1 "GND" H 7750 3830 30  0001 C CNN
 	1    7750 3900
@@
 $EndComp
 $Comp
-L GND #PWR078
+L GND #PWR077
 U 1 1 4F9A3433
 P 9100 4350
-F 0 "#PWR078" H 9100 4350 30  0001 C CNN
+F 0 "#PWR077" H 9100 4350 30  0001 C CNN
 F 1 "GND" H 9100 4280 30  0001 C CNN
 	1    9100 4350
@@
 $EndComp
 $Comp
-L GND #PWR079
+L GND #PWR078
 U 1 1 4F9A344B
 P 9950 4350
-F 0 "#PWR079" H 9950 4350 30  0001 C CNN
+F 0 "#PWR078" H 9950 4350 30  0001 C CNN
 F 1 "GND" H 9950 4280 30  0001 C CNN
 	1    9950 4350
@@
 VSS_EN
 $Comp
-L PWR_FLAG #FLG080
+L PWR_FLAG #FLG079
 U 1 1 4F9AE33C
 P 2000 3150
-F 0 "#FLG080" H 2000 3245 30  0001 C CNN
+F 0 "#FLG079" H 2000 3245 30  0001 C CNN
 F 1 "PWR_FLAG" H 2000 3330 30  0000 C CNN
 	1    2000 3150
@@
 $EndComp
 $Comp
-L PWR_FLAG #FLG081
+L PWR_FLAG #FLG080
 U 1 1 4F9AE3FD
 P 1800 3750
-F 0 "#FLG081" H 1800 3845 30  0001 C CNN
+F 0 "#FLG080" H 1800 3845 30  0001 C CNN
 F 1 "PWR_FLAG" H 1800 3930 30  0000 C CNN
 	1    1800 3750
@@
 	4400 4900 4850 4900
 Connection ~ 4850 4900
-Wire Wire Line
-	6050 4250 6050 4500
 Connection ~ 5550 4250
 Connection ~ 6050 4250
@@
 Wire Wire Line
 	9950 3750 9950 3650
-Wire Wire Line
-	10250 3150 10250 3100
-Connection ~ 10250 3150
-Connection ~ 10250 3150
 Wire Wire Line
 	2500 3800 3000 3800
@@
 Connection ~ 1800 3900
 $Comp
-L TP P9
-U 1 1 4F9AD953
-P 10250 3100
-F 0 "P9" H 10250 3450 40  0000 C CNN
-F 1 "TP" H 10250 3350 30  0001 C CNN
-F 2 "TESTVIA_p30mil_h20mil" H 10250 3100 60  0001 C CNN
-F 4 "TESTPOINT VIA" H 10250 3100 60  0001 C CNN "Description"
-F 5 "NO PART. TEST PAD ONLY." H 10250 3100 60  0001 C CNN "Note"
-F 6 "AVSS" H 10250 3350 60  0000 C CNN "Silkscreen"
-	1    10250 3100
-	1    0    0    -1
-$EndComp
-$Comp
-L SCI_AVDD_5_5V #PWR082
+L SCI_AVDD_5_5V #PWR081
 U 1 1 4F9AF0E1
 P 900 2650
-F 0 "#PWR082" H 900 2750 30  0001 C CNN
+F 0 "#PWR081" H 900 2750 30  0001 C CNN
 F 1 "SCI_AVDD_5_5V" H 900 2750 60  0000 C CNN
 	1    900  2650
